File: KiCAD/LED_clock/LED_clock.kicad_pcb (KiCad board)
At the start: 2 copper layers, 373 parts, among them U1 ICM7218A

Commit message: initial placement
Parts:
- added U1: ICM7218A, Package_DIP:DIP-28_W15.24mm_LongPads, F.Cu at (269.2, 78.7)
- added U2: ICM7218A, Package_DIP:DIP-28_W15.24mm_LongPads, F.Cu at (175.8, 115.1)
- added U3: ICM7218A, Package_DIP:DIP-28_W15.24mm_LongPads, F.Cu at (160.6, 214.1)
- added U4: ICM7218A, Package_DIP:DIP-28_W15.24mm_LongPads, F.Cu at (238.8, 276.9)
- added U5: ICM7218A, Package_DIP:DIP-28_W15.24mm_LongPads, F.Cu at (332.2, 240.5)
- moved U6 192.1 mm to (347.4, 141.5), turned to -150 degrees
- moved D116 170.4 mm to (300.0, 187.6)
- moved D121 170.4 mm to (298.7, 163.3)
- moved D167 170.4 mm to (270.5, 214.9)
- moved D171 170.4 mm to (284.2, 205.0)
- moved D189 170.4 mm to (270.5, 140.7)
- moved D226 170.4 mm to (264.6, 210.4)
- moved D235 170.4 mm to (286.6, 188.4)
- moved D238 170.4 mm to (288.3, 177.8)
- moved D241 170.4 mm to (286.6, 167.2)
- moved D250 170.4 mm to (264.6, 145.2)
- moved D251 170.4 mm to (261.1, 144.3)
- moved D276 170.4 mm to (235.3, 198.6)
- moved D290 170.4 mm to (272.7, 198.6)
- moved D300 170.4 mm to (281.3, 172.0)
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- renumbered U1 to U6
Connections:
- net Net-(D100-A) renamed /R4_X3
- net Net-(D100-K) renamed /R4_Y3
- net Net-(D101-A) renamed /R4_X4
- net Net-(D102-A) renamed /R4_X5
- net Net-(D103-A) renamed /R4_X6
- net Net-(D104-A) renamed /R4_X7
- net Net-(D105-A) renamed /R4_X0
- net Net-(D106-A) renamed /R4_X1
- net Net-(D107-A) renamed /R4_X2
- net Net-(D113-K) renamed /R4_Y5
- net Net-(D121-K) renamed /R4_Y6
- net Net-(D129-K) renamed /R4_Y7
- net Net-(D13-A) renamed /R5_X0
- net Net-(D13-K) renamed /R5_Y0
- net Net-(D133-A) renamed /R3_X0
- net Net-(D133-K) renamed /R3_Y0
- net Net-(D134-A) renamed /R3_X1
- net Net-(D135-A) renamed /R3_X2
- net Net-(D136-A) renamed /R3_X3
- net Net-(D137-A) renamed /R3_X4
- net Net-(D138-A) renamed /R3_X5
- net Net-(D139-A) renamed /R3_X6
- net Net-(D14-A) renamed /R5_X1
- net Net-(D140-A) renamed /R3_X7
- net Net-(D141-K) renamed /R3_Y1
- net Net-(D149-K) renamed /R3_Y2
- net Net-(D15-A) renamed /R5_X2
- net Net-(D157-K) renamed /R3_Y3
- net Net-(D16-A) renamed /R5_X3
- net Net-(D17-A) renamed /R5_X4
- net Net-(D173-K) renamed /R3_Y5
- net Net-(D18-A) renamed /R5_X5
- net Net-(D181-K) renamed /R3_Y6
- net Net-(D189-K) renamed /R3_Y7
- net Net-(D19-A) renamed /R5_X6
- net Net-(D193-A) renamed /R2_X0
- net Net-(D193-K) renamed /R2_Y0
- net Net-(D194-A) renamed /R2_X1
- net Net-(D195-A) renamed /R2_X2
- net Net-(D196-A) renamed /R2_X3
- net Net-(D197-A) renamed /R2_X4
- net Net-(D198-A) renamed /R2_X5
- net Net-(D199-A) renamed /R2_X6
- net Net-(D20-A) renamed /R5_X7
- net Net-(D200-A) renamed /R2_X7
- net Net-(D201-K) renamed /R2_Y1
- net Net-(D209-K) renamed /R2_Y2
- net Net-(D21-K) renamed /R5_Y1
- net Net-(D217-K) renamed /R2_Y3
- net Net-(D233-K) renamed /R2_Y5
- net Net-(D241-K) renamed /R2_Y6
- net Net-(D249-K) renamed /R2_Y7
- net Net-(D29-K) renamed /R5_Y2
- net Net-(D37-K) renamed /R5_Y3
- net Net-(D53-K) renamed /R5_Y5
- net Net-(D61-K) renamed /R5_Y6
- net Net-(D69-K) renamed /R5_Y7
- net Net-(D73-K) renamed /R4_Y0
- net Net-(D81-K) renamed /R4_Y1
- net Net-(D89-K) renamed /R4_Y2
- D105 pad 1: unconnected-(D105-K-Pad1) -> /R4_Y4
- D106 pad 1: unconnected-(D106-K-Pad1) -> /R4_Y4
- D107 pad 1: unconnected-(D107-K-Pad1) -> /R4_Y4
- D108 pad 1: unconnected-(D108-K-Pad1) -> /R4_Y4
- D109 pad 1: unconnected-(D109-K-Pad1) -> /R4_Y4
- D110 pad 1: unconnected-(D110-K-Pad1) -> /R4_Y4
- D111 pad 1: unconnected-(D111-K-Pad1) -> /R4_Y4
- D112 pad 1: unconnected-(D112-K-Pad1) -> /R4_Y4
- D165 pad 1: unconnected-(D165-K-Pad1) -> /R3_Y4
- D166 pad 1: unconnected-(D166-K-Pad1) -> /R3_Y4
- D167 pad 1: unconnected-(D167-K-Pad1) -> /R3_Y4
- D168 pad 1: unconnected-(D168-K-Pad1) -> /R3_Y4
- D169 pad 1: unconnected-(D169-K-Pad1) -> /R3_Y4
- D170 pad 1: unconnected-(D170-K-Pad1) -> /R3_Y4
- D171 pad 1: unconnected-(D171-K-Pad1) -> /R3_Y4
- D172 pad 1: unconnected-(D172-K-Pad1) -> /R3_Y4
- D225 pad 1: unconnected-(D225-K-Pad1) -> /R2_Y4
- D226 pad 1: unconnected-(D226-K-Pad1) -> /R2_Y4
- D227 pad 1: unconnected-(D227-K-Pad1) -> /R2_Y4
- D228 pad 1: unconnected-(D228-K-Pad1) -> /R2_Y4
- D229 pad 1: unconnected-(D229-K-Pad1) -> /R2_Y4
- D230 pad 1: unconnected-(D230-K-Pad1) -> /R2_Y4
- D231 pad 1: unconnected-(D231-K-Pad1) -> /R2_Y4
- D232 pad 1: unconnected-(D232-K-Pad1) -> /R2_Y4
- D253 pad 1: Net-(D253-K) -> /R1_Y0
- D253 pad 2: Net-(D253-A) -> /R1_X0
- D254 pad 1: Net-(D253-K) -> /R1_Y0
- D254 pad 2: Net-(D254-A) -> /R1_X1
- D255 pad 1: Net-(D253-K) -> /R1_Y0
- D255 pad 2: Net-(D255-A) -> /R1_X2
- D256 pad 1: Net-(D253-K) -> /R1_Y0
- D256 pad 2: Net-(D256-A) -> /R1_X3
- D257 pad 1: Net-(D253-K) -> /R1_Y0
- D257 pad 2: Net-(D257-A) -> /R1_X4
- D258 pad 1: Net-(D253-K) -> /R1_Y0
- D258 pad 2: Net-(D258-A) -> /R1_X5
- D259 pad 1: Net-(D253-K) -> /R1_Y0
- D259 pad 2: Net-(D259-A) -> /R1_X6
- D260 pad 1: Net-(D253-K) -> /R1_Y0
- D260 pad 2: Net-(D260-A) -> /R1_X7
- D261 pad 1: Net-(D261-K) -> /R1_Y1
- D261 pad 2: Net-(D253-A) -> /R1_X0
- D262 pad 1: Net-(D261-K) -> /R1_Y1
- D262 pad 2: Net-(D254-A) -> /R1_X1
- D263 pad 1: Net-(D261-K) -> /R1_Y1
- D263 pad 2: Net-(D255-A) -> /R1_X2
- D264 pad 1: Net-(D261-K) -> /R1_Y1
- D264 pad 2: Net-(D256-A) -> /R1_X3
- D265 pad 1: Net-(D261-K) -> /R1_Y1
- D265 pad 2: Net-(D257-A) -> /R1_X4
- D266 pad 1: Net-(D261-K) -> /R1_Y1
- D266 pad 2: Net-(D258-A) -> /R1_X5
- D267 pad 1: Net-(D261-K) -> /R1_Y1
- D267 pad 2: Net-(D259-A) -> /R1_X6
- D268 pad 1: Net-(D261-K) -> /R1_Y1
- D268 pad 2: Net-(D260-A) -> /R1_X7
- D269 pad 1: Net-(D269-K) -> /R1_Y2
- D269 pad 2: Net-(D253-A) -> /R1_X0
- D270 pad 1: Net-(D269-K) -> /R1_Y2
- D270 pad 2: Net-(D254-A) -> /R1_X1
- D271 pad 1: Net-(D269-K) -> /R1_Y2
- D271 pad 2: Net-(D255-A) -> /R1_X2
- D272 pad 1: Net-(D269-K) -> /R1_Y2
- D272 pad 2: Net-(D256-A) -> /R1_X3
- D273 pad 1: Net-(D269-K) -> /R1_Y2
- D273 pad 2: Net-(D257-A) -> /R1_X4
- D274 pad 1: Net-(D269-K) -> /R1_Y2
- D274 pad 2: Net-(D258-A) -> /R1_X5
- D275 pad 1: Net-(D269-K) -> /R1_Y2
- D275 pad 2: Net-(D259-A) -> /R1_X6
- D276 pad 1: Net-(D269-K) -> /R1_Y2
- D276 pad 2: Net-(D260-A) -> /R1_X7
- D277 pad 1: Net-(D277-K) -> /R1_Y3
- D277 pad 2: Net-(D253-A) -> /R1_X0
- D278 pad 1: Net-(D277-K) -> /R1_Y3
- D278 pad 2: Net-(D254-A) -> /R1_X1
- D279 pad 1: Net-(D277-K) -> /R1_Y3
- D279 pad 2: Net-(D255-A) -> /R1_X2
- D280 pad 1: Net-(D277-K) -> /R1_Y3
- D280 pad 2: Net-(D256-A) -> /R1_X3
- D281 pad 1: Net-(D277-K) -> /R1_Y3
- D281 pad 2: Net-(D257-A) -> /R1_X4
- D282 pad 1: Net-(D277-K) -> /R1_Y3
- D282 pad 2: Net-(D258-A) -> /R1_X5
- D283 pad 1: Net-(D277-K) -> /R1_Y3
- D283 pad 2: Net-(D259-A) -> /R1_X6
- D284 pad 1: Net-(D277-K) -> /R1_Y3
- D284 pad 2: Net-(D260-A) -> /R1_X7
- D285 pad 1: unconnected-(D285-K-Pad1) -> /R1_Y4
- D285 pad 2: Net-(D253-A) -> /R1_X0
- D286 pad 1: unconnected-(D286-K-Pad1) -> /R1_Y4
- D286 pad 2: Net-(D254-A) -> /R1_X1
- D287 pad 1: unconnected-(D287-K-Pad1) -> /R1_Y4
- D287 pad 2: Net-(D255-A) -> /R1_X2
- D288 pad 1: unconnected-(D288-K-Pad1) -> /R1_Y4
- D288 pad 2: Net-(D256-A) -> /R1_X3
- D289 pad 1: unconnected-(D289-K-Pad1) -> /R1_Y4
- D289 pad 2: Net-(D257-A) -> /R1_X4
- D290 pad 1: unconnected-(D290-K-Pad1) -> /R1_Y4
- D290 pad 2: Net-(D258-A) -> /R1_X5
- D291 pad 1: unconnected-(D291-K-Pad1) -> /R1_Y4
- D291 pad 2: Net-(D259-A) -> /R1_X6
- D292 pad 1: unconnected-(D292-K-Pad1) -> /R1_Y4
- D292 pad 2: Net-(D260-A) -> /R1_X7
- D293 pad 1: Net-(D293-K) -> /R1_Y5
- D293 pad 2: Net-(D253-A) -> /R1_X0
- D294 pad 1: Net-(D293-K) -> /R1_Y5
- D294 pad 2: Net-(D254-A) -> /R1_X1
- D295 pad 1: Net-(D293-K) -> /R1_Y5
- D295 pad 2: Net-(D255-A) -> /R1_X2
- D296 pad 1: Net-(D293-K) -> /R1_Y5
- D296 pad 2: Net-(D256-A) -> /R1_X3
- D297 pad 1: Net-(D293-K) -> /R1_Y5
- D297 pad 2: Net-(D257-A) -> /R1_X4
- D298 pad 1: Net-(D293-K) -> /R1_Y5
- D298 pad 2: Net-(D258-A) -> /R1_X5
- D299 pad 1: Net-(D293-K) -> /R1_Y5
- D299 pad 2: Net-(D259-A) -> /R1_X6
- D300 pad 1: Net-(D293-K) -> /R1_Y5
- D300 pad 2: Net-(D260-A) -> /R1_X7
- D301 pad 1: Net-(D301-K) -> /R1_Y6
- D301 pad 2: Net-(D253-A) -> /R1_X0
- D302 pad 1: Net-(D301-K) -> /R1_Y6
- D302 pad 2: Net-(D254-A) -> /R1_X1
- D303 pad 1: Net-(D301-K) -> /R1_Y6
- D303 pad 2: Net-(D255-A) -> /R1_X2
- D304 pad 1: Net-(D301-K) -> /R1_Y6
- D304 pad 2: Net-(D256-A) -> /R1_X3
- D305 pad 1: Net-(D301-K) -> /R1_Y6
- D305 pad 2: Net-(D257-A) -> /R1_X4
- D306 pad 1: Net-(D301-K) -> /R1_Y6
- D306 pad 2: Net-(D258-A) -> /R1_X5
- D307 pad 1: Net-(D301-K) -> /R1_Y6
- D307 pad 2: Net-(D259-A) -> /R1_X6
- D308 pad 1: Net-(D301-K) -> /R1_Y6
- D308 pad 2: Net-(D260-A) -> /R1_X7
- D309 pad 1: Net-(D309-K) -> /R1_Y7
- D309 pad 2: Net-(D253-A) -> /R1_X0
- D310 pad 1: Net-(D309-K) -> /R1_Y7
- D310 pad 2: Net-(D254-A) -> /R1_X1
- D311 pad 1: Net-(D309-K) -> /R1_Y7
- D311 pad 2: Net-(D255-A) -> /R1_X2
- D312 pad 1: Net-(D309-K) -> /R1_Y7
- D312 pad 2: Net-(D256-A) -> /R1_X3
- D45 pad 1: unconnected-(D45-K-Pad1) -> /R5_Y4
- D46 pad 1: unconnected-(D46-K-Pad1) -> /R5_Y4
- D47 pad 1: unconnected-(D47-K-Pad1) -> /R5_Y4
- D48 pad 1: unconnected-(D48-K-Pad1) -> /R5_Y4
- D49 pad 1: unconnected-(D49-K-Pad1) -> /R5_Y4
- D50 pad 1: unconnected-(D50-K-Pad1) -> /R5_Y4
- D51 pad 1: unconnected-(D51-K-Pad1) -> /R5_Y4
- D52 pad 1: unconnected-(D52-K-Pad1) -> /R5_Y4
- U6 pad 1: /R7_Y2 -> /R1_Y2
- U6 pad 15: /R7_X0 -> /R1_X0
- U6 pad 16: /R7_X1 -> /R1_X1
- U6 pad 17: /R7_X4 -> /R1_X4
- U6 pad 18: /R7_X7 -> /R1_X7
- U6 pad 19: unconnected-(U1-V+-Pad19) -> VCC
- U6 pad 2: /R7_Y4 -> /R1_Y4
- U6 pad 20: /R7_X3 -> /R1_X3
- U6 pad 21: /R7_X6 -> /R1_X6
- U6 pad 22: /R7_X5 -> /R1_X5
- U6 pad 23: /R7_X2 -> /R1_X2
- U6 pad 24: /R7_Y5 -> /R1_Y5
- U6 pad 25: /R7_Y3 -> /R1_Y3
- U6 pad 26: /R7_Y6 -> /R1_Y6
- U6 pad 27: /R7_Y0 -> /R1_Y0
- U6 pad 28: unconnected-(U1-GND-Pad28) -> GND
- U6 pad 3: /R7_Y1 -> /R1_Y1
- U6 pad 4: /R7_Y7 -> /R1_Y7
Other:
- board outline added: 228.6 x 228.6 mm
