File: KiCAD/LED_clock/LED_clock.kicad_pcb (KiCad board)
At the start: 2 copper layers, 228.6 x 228.6 mm, 392 parts, among them J1 CONN_2X10, U1 ICM7218A, U2 ICM7218A, U3 ICM7218A, U4 ICM7218A, U5 ICM7218A, U6 ICM7218A, U7 74HC138, U8 74LS244, U9 74LS125

Commit message: tentative placement
Parts:
- removed the D12 at (284.9, 124.4)
- removed the D132 at (258.9, 131.1)
- removed the D192 at (258.2, 137.4)
- removed the D252 at (257.6, 143.7)
- removed the D312 at (256.9, 150.0)
- removed the D372 at (261.4, 107.8)
- removed the D72 at (259.7, 123.5)
- removed the U6 at (347.4, 141.5)
- added D1: LED, LED_THT:LED_D5.0mm, F.Cu at (254.0, 77.5)
- added D13: LED, LED_THT:LED_D3.0mm, F.Cu at (254.0, 83.8)
- added D133: LED, LED_SMD:LED_1206_3216Metric_Pad1.42x1.75mm_HandSolder, F.Cu at (254.0, 101.6)
- added D193: LED, LED_SMD:LED_1206_3216Metric_Pad1.42x1.75mm_HandSolder, F.Cu at (254.0, 114.1)
- added D253: LED, LED_SMD:LED_1206_3216Metric_Pad1.42x1.75mm_HandSolder, F.Cu at (254.0, 127.0)
- added D313: LED, LED_THT:LED_D3.0mm, F.Cu at (254.0, 71.1)
- added D73: LED, LED_SMD:LED_1206_3216Metric_Pad1.42x1.75mm_HandSolder, F.Cu at (254.0, 88.9)
- added U1: ICM7218A, Package_LCC:PLCC-28, F.Cu at (254.0, 142.2)
- C1, C2, C6: footprint Capacitor_THT:C_Disc_D4.3mm_W1.9mm_P5.00mm -> Capacitor_SMD:C_1206_3216Metric_Pad1.33x1.80mm_HandSolder
- C3, C4, C5, C7, C8, C9: footprint Capacitor_THT:C_Disc_D4.3mm_W1.9mm_P5.00mm -> Capacitor_SMD:C_1206_3216Metric_Pad1.33x1.80mm_HandSolder; moved to B.Cu
- J1: moved to B.Cu
- U2, U3, U4, U5: footprint Package_DIP:DIP-28_W15.24mm_LongPads -> Package_LCC:PLCC-28
- U6: renamed from U1; footprint Package_DIP:DIP-28_W15.24mm_LongPads -> Package_LCC:PLCC-28
- U7: footprint Package_DIP:DIP-16_W7.62mm_LongPads -> Package_SO:SO-16_3.9x9.9mm_P1.27mm
- U8: footprint Package_DIP:DIP-20_W7.62mm_LongPads -> Package_SO:SO-20_5.3x12.6mm_P1.27mm
- U9: footprint Package_DIP:DIP-14_W7.62mm_LongPads -> Package_SO:SO-14_3.9x8.65mm_P1.27mm
- moved C5 124.2 mm to (253.7, 142.2), turned to 180 degrees
- moved C3 123.6 mm to (284.8, 195.6), turned to 180 degrees
- moved C7 109.9 mm to (223.5, 160.0), turned to 180 degrees
- moved C8 106.4 mm to (284.8, 160.0), turned to 180 degrees
- moved C2 104.2 mm to (269.5, 171.4), turned to 180 degrees
- moved U7 99.0 mm to (236.2, 178.4), turned to 0 degrees
- moved U8 98.3 mm to (253.1, 178.4), turned to 0 degrees
- moved J1 96.2 mm to (264.2, 194.3)
- moved C6 95.7 mm to (253.7, 168.9), turned to 180 degrees
- moved C1 94.5 mm to (236.5, 170.2), turned to 180 degrees
- moved C10 85.4 mm to (253.3, 200.7)
- moved U6 82.8 mm to (284.8, 160.0), turned to 30 degrees
- moved U9 81.3 mm to (269.2, 179.1), turned to 0 degrees
- moved C9 74.6 mm to (223.5, 195.6), turned to 180 degrees
- moved U4 65.3 mm to (254.0, 213.4), turned to -90 degrees
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- renumbered D1 to D12, D73 to D132, D133 to D192, D193 to D252, D253 to D312, D313 to D372, D13 to D72
Connections:
- D12 pad 1: /R7_X4 -> /R4_X7
- D12 pad 2: /R7_Y6 -> /R4_Y6
- D132 pad 1: /R4_Y0 -> /R4_Y7
- D132 pad 2: /R4_X0 -> /R4_X3
- D192 pad 1: /R3_Y0 -> /R3_Y7
- D192 pad 2: /R3_X0 -> /R3_X3
- D252 pad 1: /R2_Y0 -> /R2_Y7
- D252 pad 2: /R2_X0 -> /R2_X3
- D312 pad 1: /R1_Y0 -> /R1_Y7
- D312 pad 2: /R1_X0 -> /R1_X3
- D372 pad 1: /R7_Y0 -> /R7_Y7
- D372 pad 2: /R7_X0 -> /R7_X3
- D72 pad 1: /R5_Y0 -> /R5_Y7
- D72 pad 2: /R5_X0 -> /R5_X3
- U2 pad 1: /R5_Y2 -> /R7_Y2
- U2 pad 15: /R5_X0 -> /R7_X0
- U2 pad 16: /R5_X1 -> /R7_X1
- U2 pad 17: /R5_X4 -> /R7_X4
- U2 pad 18: /R5_X7 -> /R7_X7
- U2 pad 2: /R5_Y4 -> /R7_Y4
- U2 pad 20: /R5_X3 -> /R7_X3
- U2 pad 21: /R5_X6 -> /R7_X6
- U2 pad 22: /R5_X5 -> /R7_X5
- U2 pad 23: /R5_X2 -> /R7_X2
- U2 pad 24: /R5_Y5 -> /R7_Y5
- U2 pad 25: /R5_Y3 -> /R7_Y3
- U2 pad 26: /R5_Y6 -> /R7_Y6
- U2 pad 27: /R5_Y0 -> /R7_Y0
- U2 pad 3: /R5_Y1 -> /R7_Y1
- U2 pad 4: /R5_Y7 -> /R7_Y7
- U2 pad 8: /~{RING5} -> /~{RING7}
- U3 pad 1: /R4_Y2 -> /R7_Y2
- U3 pad 15: /R4_X0 -> /R7_X0
- U3 pad 16: /R4_X1 -> /R7_X1
- U3 pad 17: /R4_X4 -> /R7_X4
- U3 pad 18: /R4_X7 -> /R7_X7
- U3 pad 2: /R4_Y4 -> /R7_Y4
- U3 pad 20: /R4_X3 -> /R7_X3
- U3 pad 21: /R4_X6 -> /R7_X6
- U3 pad 22: /R4_X5 -> /R7_X5
- U3 pad 23: /R4_X2 -> /R7_X2
- U3 pad 24: /R4_Y5 -> /R7_Y5
- U3 pad 25: /R4_Y3 -> /R7_Y3
- U3 pad 26: /R4_Y6 -> /R7_Y6
- U3 pad 27: /R4_Y0 -> /R7_Y0
- U3 pad 3: /R4_Y1 -> /R7_Y1
- U3 pad 4: /R4_Y7 -> /R7_Y7
- U3 pad 8: /~{RING4} -> /~{RING7}
- U4 pad 1: /R3_Y2 -> /R7_Y2
- U4 pad 15: /R3_X0 -> /R7_X0
- U4 pad 16: /R3_X1 -> /R7_X1
- U4 pad 17: /R3_X4 -> /R7_X4
- U4 pad 18: /R3_X7 -> /R7_X7
- U4 pad 2: /R3_Y4 -> /R7_Y4
- U4 pad 20: /R3_X3 -> /R7_X3
- U4 pad 21: /R3_X6 -> /R7_X6
- U4 pad 22: /R3_X5 -> /R7_X5
- U4 pad 23: /R3_X2 -> /R7_X2
- U4 pad 24: /R3_Y5 -> /R7_Y5
- U4 pad 25: /R3_Y3 -> /R7_Y3
- U4 pad 26: /R3_Y6 -> /R7_Y6
- U4 pad 27: /R3_Y0 -> /R7_Y0
- U4 pad 3: /R3_Y1 -> /R7_Y1
- U4 pad 4: /R3_Y7 -> /R7_Y7
- U4 pad 8: /~{RING3} -> /~{RING7}
- U5 pad 1: /R2_Y2 -> /R7_Y2
- U5 pad 15: /R2_X0 -> /R7_X0
- U5 pad 16: /R2_X1 -> /R7_X1
- U5 pad 17: /R2_X4 -> /R7_X4
- U5 pad 18: /R2_X7 -> /R7_X7
- U5 pad 2: /R2_Y4 -> /R7_Y4
- U5 pad 20: /R2_X3 -> /R7_X3
- U5 pad 21: /R2_X6 -> /R7_X6
- U5 pad 22: /R2_X5 -> /R7_X5
- U5 pad 23: /R2_X2 -> /R7_X2
- U5 pad 24: /R2_Y5 -> /R7_Y5
- U5 pad 25: /R2_Y3 -> /R7_Y3
- U5 pad 26: /R2_Y6 -> /R7_Y6
- U5 pad 27: /R2_Y0 -> /R7_Y0
- U5 pad 3: /R2_Y1 -> /R7_Y1
- U5 pad 4: /R2_Y7 -> /R7_Y7
- U5 pad 8: /~{RING2} -> /~{RING7}
Other:
- copper layers 2 -> 4
