File: KiCAD/LED_clock/LED_clock.kicad_sch (KiCad schematic)
At the start: 373 parts, among them U1 ICM7218A

Commit message: initial placement
Parts:
- added U2, U3, U4, U5, U6: ICM7218A, Package_DIP:DIP-28_W15.24mm_LongPads, symbol ICM7218A:ICM7218A
Connections:
- net GND: now also U2.28 (GND), U3.28 (GND), U4.28 (GND), U5.28 (GND), U6.28 (GND)
- net VCC: now also U2.19 (V+), U3.19 (V+), U4.19 (V+), U5.19 (V+), U6.19 (V+)
- net R2_Y2: now reaches D209.1 (K), D210.1 (K), D211.1 (K), D212.1 (K), D213.1 (K), D214.1 (K), D215.1 (K), D216.1 (K)
- net R2_Y2: now also U5.1 (c)
- net R2_X7: now reaches D200.2 (A), D208.2 (A), D216.2 (A), D224.2 (A), D232.2 (A), D240.2 (A), D248.2 (A)
- net R2_X7: now also U5.18 (d8)
- net R1_Y6: now reaches D301.1 (K), D302.1 (K), D303.1 (K), D304.1 (K), D305.1 (K), D306.1 (K), D307.1 (K), D308.1 (K)
- net R1_Y6: now also U6.26 (g)
- net R1_X7: now reaches D260.2 (A), D268.2 (A), D276.2 (A), D284.2 (A), D292.2 (A), D300.2 (A), D308.2 (A)
- net R1_X7: now also U6.18 (d8)
- net R2_Y1: now reaches D201.1 (K), D202.1 (K), D203.1 (K), D204.1 (K), D205.1 (K), D206.1 (K), D207.1 (K), D208.1 (K)
- net R2_Y1: now also U5.3 (b)
- net R2_X2: now reaches D195.2 (A), D203.2 (A), D211.2 (A), D219.2 (A), D227.2 (A), D235.2 (A), D243.2 (A), D251.2 (A)
- net R2_X2: now also U5.23 (d3)
- net R1_Y1: now reaches D261.1 (K), D262.1 (K), D263.1 (K), D264.1 (K), D265.1 (K), D266.1 (K), D267.1 (K), D268.1 (K)
- net R1_Y1: now also U6.3 (b)
- net R1_X0: now reaches D253.2 (A), D261.2 (A), D269.2 (A), D277.2 (A), D285.2 (A), D293.2 (A), D301.2 (A), D309.2 (A)
- net R1_X0: now also U6.15 (d1)
- net R5_Y6: now reaches D61.1 (K), D62.1 (K), D63.1 (K), D64.1 (K), D65.1 (K), D66.1 (K), D67.1 (K), D68.1 (K)
- net R5_Y6: now also U2.26 (g)
- net R5_X7: now reaches D20.2 (A), D28.2 (A), D36.2 (A), D44.2 (A), D52.2 (A), D60.2 (A), D68.2 (A)
- net R5_X7: now also U2.18 (d8)
- net R4_Y0: now reaches D73.1 (K), D74.1 (K), D75.1 (K), D76.1 (K), D77.1 (K), D78.1 (K), D79.1 (K), D80.1 (K)
- net R4_Y0: now also U3.27 (a)
- net R4_X7: now reaches D104.2 (A), D112.2 (A), D120.2 (A), D128.2 (A), D80.2 (A), D88.2 (A), D96.2 (A)
- net R4_X7: now also U3.18 (d8)
- net R5_Y4: now reaches D50.1 (K)
- net R5_Y4: now also D45.1 (K), D46.1 (K), D47.1 (K), D48.1 (K), D49.1 (K), D51.1 (K), D52.1 (K), U2.2 (e)
- net R5_X5: now reaches D18.2 (A), D26.2 (A), D34.2 (A), D42.2 (A), D50.2 (A), D58.2 (A), D66.2 (A)
- net R5_X5: now also U2.22 (d6)
- net R5_Y2: now reaches D29.1 (K), D30.1 (K), D31.1 (K), D32.1 (K), D33.1 (K), D34.1 (K), D35.1 (K), D36.1 (K)
- net R5_Y2: now also U2.1 (c)
- net R3_Y7: now reaches D189.1 (K), D190.1 (K), D191.1 (K), D192.1 (K)
- net R3_Y7: now also U4.4 (dp)
- net R3_X1: now reaches D134.2 (A), D142.2 (A), D150.2 (A), D158.2 (A), D166.2 (A), D174.2 (A), D182.2 (A), D190.2 (A)
- net R3_X1: now also U4.16 (d2)
- net R4_Y4: now reaches D107.1 (K)
- net R4_Y4: now also D105.1 (K), D106.1 (K), D108.1 (K), D109.1 (K), D110.1 (K), D111.1 (K), D112.1 (K), U3.2 (e)
- net R4_X2: now reaches D107.2 (A), D115.2 (A), D123.2 (A), D131.2 (A), D75.2 (A), D83.2 (A), D91.2 (A), D99.2 (A)
- net R4_X2: now also U3.23 (d3)
- net R2_Y7: now reaches D249.1 (K), D250.1 (K), D251.1 (K), D252.1 (K)
- net R2_Y7: now also U5.4 (dp)
- net R2_X1: now reaches D194.2 (A), D202.2 (A), D210.2 (A), D218.2 (A), D226.2 (A), D234.2 (A), D242.2 (A), D250.2 (A)
- net R2_X1: now also U5.16 (d2)
- net R2_Y3: now reaches D217.1 (K), D218.1 (K), D219.1 (K), D220.1 (K), D221.1 (K), D222.1 (K), D223.1 (K), D224.1 (K)
- net R2_Y3: now also U5.25 (d)
- net R2_Y0: now reaches D193.1 (K), D194.1 (K), D195.1 (K), D196.1 (K), D197.1 (K), D198.1 (K), D199.1 (K), D200.1 (K)
- net R2_Y0: now also U5.27 (a)
- net R1_X3: now reaches D256.2 (A), D264.2 (A), D272.2 (A), D280.2 (A), D288.2 (A), D296.2 (A), D304.2 (A), D312.2 (A)
- net R1_X3: now also U6.20 (d4)
- net R4_X0: now reaches D105.2 (A), D113.2 (A), D121.2 (A), D129.2 (A), D73.2 (A), D81.2 (A), D89.2 (A), D97.2 (A)
- net R4_X0: now also U3.15 (d1)
- net R3_Y0: now reaches D133.1 (K), D134.1 (K), D135.1 (K), D136.1 (K), D137.1 (K), D138.1 (K), D139.1 (K), D140.1 (K)
- net R3_Y0: now also U4.27 (a)
- net R3_X0: now reaches D133.2 (A), D141.2 (A), D149.2 (A), D157.2 (A), D165.2 (A), D173.2 (A), D181.2 (A), D189.2 (A)
- net R3_X0: now also U4.15 (d1)
- net R5_X0: now reaches D13.2 (A), D21.2 (A), D29.2 (A), D37.2 (A), D45.2 (A), D53.2 (A), D61.2 (A), D69.2 (A)
- net R5_X0: now also U2.15 (d1)
- net R4_Y2: now reaches D89.1 (K), D90.1 (K), D91.1 (K), D92.1 (K), D93.1 (K), D94.1 (K), D95.1 (K), D96.1 (K)
- net R4_Y2: now also U3.1 (c)
- net R4_X4: now reaches D101.2 (A), D109.2 (A), D117.2 (A), D125.2 (A), D77.2 (A), D85.2 (A), D93.2 (A)
- net R4_X4: now also U3.17 (d5)
- net R4_Y6: now reaches D121.1 (K), D122.1 (K), D123.1 (K), D124.1 (K), D125.1 (K), D126.1 (K), D127.1 (K), D128.1 (K)
- net R4_Y6: now also U3.26 (g)
- net R4_X1: now reaches D106.2 (A), D114.2 (A), D122.2 (A), D130.2 (A), D74.2 (A), D82.2 (A), D90.2 (A), D98.2 (A)
- net R4_X1: now also U3.16 (d2)
- net R1_Y2: now reaches D269.1 (K), D270.1 (K), D271.1 (K), D272.1 (K), D273.1 (K), D274.1 (K), D275.1 (K), D276.1 (K)
- net R1_Y2: now also U6.1 (c)
- net R1_X5: now reaches D258.2 (A), D266.2 (A), D274.2 (A), D282.2 (A), D290.2 (A), D298.2 (A), D306.2 (A)
- net R1_X5: now also U6.22 (d6)
- net R2_Y5: now reaches D233.1 (K), D234.1 (K), D235.1 (K), D236.1 (K), D237.1 (K), D238.1 (K), D239.1 (K), D240.1 (K)
- net R2_Y5: now also U5.24 (f)
- net R2_X6: now reaches D199.2 (A), D207.2 (A), D215.2 (A), D223.2 (A), D231.2 (A), D239.2 (A), D247.2 (A)
- net R2_X6: now also U5.21 (d7)
- net R3_Y1: now reaches D141.1 (K), D142.1 (K), D143.1 (K), D144.1 (K), D145.1 (K), D146.1 (K), D147.1 (K), D148.1 (K)
- net R3_Y1: now also U4.3 (b)
- net R3_X3: now reaches D136.2 (A), D144.2 (A), D152.2 (A), D160.2 (A), D168.2 (A), D176.2 (A), D184.2 (A), D192.2 (A)
- net R3_X3: now also U4.20 (d4)
- net R4_Y7: now reaches D129.1 (K), D130.1 (K), D131.1 (K), D132.1 (K)
- net R4_Y7: now also U3.4 (dp)
- net R4_X3: now reaches D100.2 (A), D108.2 (A), D116.2 (A), D124.2 (A), D132.2 (A), D76.2 (A), D84.2 (A), D92.2 (A)
- net R4_X3: now also U3.20 (d4)
- net R2_X5: now reaches D198.2 (A), D206.2 (A), D214.2 (A), D222.2 (A), D230.2 (A), D238.2 (A), D246.2 (A)
- net R2_X5: now also U5.22 (d6)
- net R1_Y4: now reaches D287.1 (K)
- net R1_Y4: now also D285.1 (K), D286.1 (K), D288.1 (K), D289.1 (K), D290.1 (K), D291.1 (K), D292.1 (K), U6.2 (e)
- net R1_X2: now reaches D255.2 (A), D263.2 (A), D271.2 (A), D279.2 (A), D287.2 (A), D295.2 (A), D303.2 (A), D311.2 (A)
- net R1_X2: now also U6.23 (d3)
- net R5_Y7: now reaches D69.1 (K), D70.1 (K), D71.1 (K), D72.1 (K)
- net R5_Y7: now also U2.4 (dp)
- net R1_Y7: now reaches D309.1 (K), D310.1 (K), D311.1 (K), D312.1 (K)
- net R1_Y7: now also U6.4 (dp)
- net R4_Y1: now reaches D81.1 (K), D82.1 (K), D83.1 (K), D84.1 (K), D85.1 (K), D86.1 (K), D87.1 (K), D88.1 (K)
- net R4_Y1: now also U3.3 (b)
- net R4_X5: now reaches D102.2 (A), D110.2 (A), D118.2 (A), D126.2 (A), D78.2 (A), D86.2 (A), D94.2 (A)
- net R4_X5: now also U3.22 (d6)
- net R2_X4: now reaches D197.2 (A), D205.2 (A), D213.2 (A), D221.2 (A), D229.2 (A), D237.2 (A), D245.2 (A)
- net R2_X4: now also U5.17 (d5)
- net R5_X6: now reaches D19.2 (A), D27.2 (A), D35.2 (A), D43.2 (A), D51.2 (A), D59.2 (A), D67.2 (A)
- net R5_X6: now also U2.21 (d7)
- net R4_Y3: now reaches D100.1 (K), D101.1 (K), D102.1 (K), D103.1 (K), D104.1 (K), D97.1 (K), D98.1 (K), D99.1 (K)
- net R4_Y3: now also U3.25 (d)
- net R4_X6: now reaches D103.2 (A), D111.2 (A), D119.2 (A), D127.2 (A), D79.2 (A), D87.2 (A), D95.2 (A)
- net R4_X6: now also U3.21 (d7)
- net R3_Y2: now reaches D149.1 (K), D150.1 (K), D151.1 (K), D152.1 (K), D153.1 (K), D154.1 (K), D155.1 (K), D156.1 (K)
- net R3_Y2: now also U4.1 (c)
- net R1_Y0: now reaches D253.1 (K), D254.1 (K), D255.1 (K), D256.1 (K), D257.1 (K), D258.1 (K), D259.1 (K), D260.1 (K)
- net R1_Y0: now also U6.27 (a)
- net R3_X2: now reaches D135.2 (A), D143.2 (A), D151.2 (A), D159.2 (A), D167.2 (A), D175.2 (A), D183.2 (A), D191.2 (A)
- net R3_X2: now also U4.23 (d3)
- net R3_Y4: now reaches D170.1 (K)
- net R3_Y4: now also D165.1 (K), D166.1 (K), D167.1 (K), D168.1 (K), D169.1 (K), D171.1 (K), D172.1 (K), U4.2 (e)
- net R3_X5: now reaches D138.2 (A), D146.2 (A), D154.2 (A), D162.2 (A), D170.2 (A), D178.2 (A), D186.2 (A)
- net R3_X5: now also U4.22 (d6)
- net R2_X3: now reaches D196.2 (A), D204.2 (A), D212.2 (A), D220.2 (A), D228.2 (A), D236.2 (A), D244.2 (A), D252.2 (A)
- net R2_X3: now also U5.20 (d4)
- net R3_Y6: now reaches D181.1 (K), D182.1 (K), D183.1 (K), D184.1 (K), D185.1 (K), D186.1 (K), D187.1 (K), D188.1 (K)
- net R3_Y6: now also U4.26 (g)
- net R1_X4: now reaches D257.2 (A), D265.2 (A), D273.2 (A), D281.2 (A), D289.2 (A), D297.2 (A), D305.2 (A)
- net R1_X4: now also U6.17 (d5)
- net R2_X0: now reaches D193.2 (A), D201.2 (A), D209.2 (A), D217.2 (A), D225.2 (A), D233.2 (A), D241.2 (A), D249.2 (A)
- net R2_X0: now also U5.15 (d1)
- net R5_X3: now reaches D16.2 (A), D24.2 (A), D32.2 (A), D40.2 (A), D48.2 (A), D56.2 (A), D64.2 (A), D72.2 (A)
- net R5_X3: now also U2.20 (d4)
- net R1_Y5: now reaches D293.1 (K), D294.1 (K), D295.1 (K), D296.1 (K), D297.1 (K), D298.1 (K), D299.1 (K), D300.1 (K)
- net R1_Y5: now also U6.24 (f)
- net R5_Y0: now reaches D13.1 (K), D14.1 (K), D15.1 (K), D16.1 (K), D17.1 (K), D18.1 (K), D19.1 (K), D20.1 (K)
- net R5_Y0: now also U2.27 (a)
- net R5_Y1: now reaches D21.1 (K), D22.1 (K), D23.1 (K), D24.1 (K), D25.1 (K), D26.1 (K), D27.1 (K), D28.1 (K)
- net R5_Y1: now also U2.3 (b)
- net R3_Y5: now reaches D173.1 (K), D174.1 (K), D175.1 (K), D176.1 (K), D177.1 (K), D178.1 (K), D179.1 (K), D180.1 (K)
- net R3_Y5: now also U4.24 (f)
- net R3_X7: now reaches D140.2 (A), D148.2 (A), D156.2 (A), D164.2 (A), D172.2 (A), D180.2 (A), D188.2 (A)
- net R3_X7: now also U4.18 (d8)
- net R1_X6: now reaches D259.2 (A), D267.2 (A), D275.2 (A), D283.2 (A), D291.2 (A), D299.2 (A), D307.2 (A)
- net R1_X6: now also U6.21 (d7)
- net R5_Y3: now reaches D37.1 (K), D38.1 (K), D39.1 (K), D40.1 (K), D41.1 (K), D42.1 (K), D43.1 (K), D44.1 (K)
- net R5_Y3: now also U2.25 (d)
- net R4_Y5: now reaches D113.1 (K), D114.1 (K), D115.1 (K), D116.1 (K), D117.1 (K), D118.1 (K), D119.1 (K), D120.1 (K)
- net R4_Y5: now also U3.24 (f)
- net R5_X2: now reaches D15.2 (A), D23.2 (A), D31.2 (A), D39.2 (A), D47.2 (A), D55.2 (A), D63.2 (A), D71.2 (A)
- net R5_X2: now also U2.23 (d3)
- net R3_Y3: now reaches D157.1 (K), D158.1 (K), D159.1 (K), D160.1 (K), D161.1 (K), D162.1 (K), D163.1 (K), D164.1 (K)
- net R3_Y3: now also U4.25 (d)
- net R5_Y5: now reaches D53.1 (K), D54.1 (K), D55.1 (K), D56.1 (K), D57.1 (K), D58.1 (K), D59.1 (K), D60.1 (K)
- net R5_Y5: now also U2.24 (f)
- net R5_X4: now reaches D17.2 (A), D25.2 (A), D33.2 (A), D41.2 (A), D49.2 (A), D57.2 (A), D65.2 (A)
- net R5_X4: now also U2.17 (d5)
- net R1_Y3: now reaches D277.1 (K), D278.1 (K), D279.1 (K), D280.1 (K), D281.1 (K), D282.1 (K), D283.1 (K), D284.1 (K)
- net R1_Y3: now also U6.25 (d)
- net R1_X1: now reaches D254.2 (A), D262.2 (A), D270.2 (A), D278.2 (A), D286.2 (A), D294.2 (A), D302.2 (A), D310.2 (A)
- net R1_X1: now also U6.16 (d2)
- net R2_Y6: now reaches D241.1 (K), D242.1 (K), D243.1 (K), D244.1 (K), D245.1 (K), D246.1 (K), D247.1 (K), D248.1 (K)
- net R2_Y6: now also U5.26 (g)
- net R2_Y4: now reaches D230.1 (K)
- net R2_Y4: now also D225.1 (K), D226.1 (K), D227.1 (K), D228.1 (K), D229.1 (K), D231.1 (K), D232.1 (K), U5.2 (e)
- net R3_X4: now reaches D137.2 (A), D145.2 (A), D153.2 (A), D161.2 (A), D169.2 (A), D177.2 (A), D185.2 (A)
- net R3_X4: now also U4.17 (d5)
- net R5_X1: now reaches D14.2 (A), D22.2 (A), D30.2 (A), D38.2 (A), D46.2 (A), D54.2 (A), D62.2 (A), D70.2 (A)
- net R5_X1: now also U2.16 (d2)
- net R3_X6: now reaches D139.2 (A), D147.2 (A), D155.2 (A), D163.2 (A), D171.2 (A), D179.2 (A), D187.2 (A)
- net R3_X6: now also U4.21 (d7)
Other:
- moved on the sheet: D1, D10, D100, D101, D102, D103, D104, D105, D106, D107, D108, D109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
