File: KiCAD/LED_clock_display/LED_clock_display.kicad_sch (KiCad schematic)
At the start: 392 parts, among them J1 CONN_2X10, U1 ICM7218A, U2 ICM7218A, U3 ICM7218A, U4 ICM7218A, U5 ICM7218A, U6 ICM7218A, U7 74HC138, U8 74LS244, U9 74LS125

Commit message: Split into two boards
Parts:
- removed C1, C2, C3, C4, C5, C6, C7, C8, C9: 0.1uF, Capacitor_THT:C_Disc_D4.3mm_W1.9mm_P5.00mm, symbol Device:C
- removed C10: 33uF, Capacitor_THT:CP_Radial_D5.0mm_P2.00mm, symbol Device:C_Polarized
- removed J1: CONN_2X10, Connector_PinHeader_2.54mm:PinHeader_2x10_P2.54mm_Vertical, symbol Connector_Generic:Conn_02x10_Counter_Clockwise
- removed U1, U2, U3, U4, U5, U6: ICM7218A, Package_DIP:DIP-28_W15.24mm_LongPads, symbol ICM7218A:ICM7218A
- removed U7: 74HC138, Package_DIP:DIP-16_W7.62mm_LongPads, symbol 74xx:74HC138
- removed U8: 74LS244, Package_DIP:DIP-20_W7.62mm_LongPads, symbol 74xx:74LS244
- removed U9: 74LS125, Package_DIP:DIP-14_W7.62mm_LongPads, symbol 74xx:74LS125
- added J1, J10, J11, J12, J13, J14, J15, J16, J17, J18, J19, J2, J20, J21, J22, J23, J24, J25, J26, J27, J28, J29, J3, J30, J31, J32, J33, J34, J35, J36, J37, J38, J39, J4, J40, J41, J42, J43, J44, J45, J46, J47, J48, J49, J5, J50, J51, J52, J53, J54, J55, J56, J57, J58, J59, J6, J60, J61, J62, J63, J64, J65, J66, J67, J68, J69, J7, J70, J71, J72, J73, J74, J75, J76, J77, J78, J79, J8, J80, J81, J82, J83, J84, J85, J86, J87, J88, J89, J9, J90, J91, J92, J93, J94, J95, J96: PIN, TestPoint:TestPoint_THTPad_D2.0mm_Drill1.0mm, symbol Connector:Conn_01x01_Pin
Connections:
- net R1_X0: now also J81.1 (Pin_1)
- net R1_X1: now also J82.1 (Pin_1)
- net R1_X2: now also J83.1 (Pin_1)
- net R1_X3: now also J84.1 (Pin_1)
- net R1_X4: now also J85.1 (Pin_1)
- net R1_X5: now also J86.1 (Pin_1)
- net R1_X6: now also J87.1 (Pin_1)
- net R1_X7: now also J88.1 (Pin_1)
- net R1_Y0: now also J89.1 (Pin_1)
- net R1_Y1: now also J90.1 (Pin_1)
- net R1_Y2: now also J91.1 (Pin_1)
- net R1_Y3: now also J92.1 (Pin_1)
- net R1_Y4: now also J93.1 (Pin_1)
- net R1_Y5: now also J94.1 (Pin_1)
- net R1_Y6: now also J95.1 (Pin_1)
- net R1_Y7: now also J96.1 (Pin_1)
- net R2_X0: now also J65.1 (Pin_1)
- net R2_X1: now also J66.1 (Pin_1)
- net R2_X2: now also J67.1 (Pin_1)
- net R2_X3: now also J68.1 (Pin_1)
- net R2_X4: now also J69.1 (Pin_1)
- net R2_X5: now also J70.1 (Pin_1)
- net R2_X6: now also J71.1 (Pin_1)
- net R2_X7: now also J72.1 (Pin_1)
- net R2_Y0: now also J73.1 (Pin_1)
- net R2_Y1: now also J74.1 (Pin_1)
- net R2_Y2: now also J75.1 (Pin_1)
- net R2_Y3: now also J76.1 (Pin_1)
- net R2_Y4: now also J77.1 (Pin_1)
- net R2_Y5: now also J78.1 (Pin_1)
- net R2_Y6: now also J79.1 (Pin_1)
- net R2_Y7: now also J80.1 (Pin_1)
- net R3_X0: now also J49.1 (Pin_1)
- net R3_X1: now also J50.1 (Pin_1)
- net R3_X2: now also J51.1 (Pin_1)
- net R3_X3: now also J52.1 (Pin_1)
- net R3_X4: now also J53.1 (Pin_1)
- net R3_X5: now also J54.1 (Pin_1)
- net R3_X6: now also J55.1 (Pin_1)
- net R3_X7: now also J56.1 (Pin_1)
- net R3_Y0: now also J57.1 (Pin_1)
- net R3_Y1: now also J58.1 (Pin_1)
- net R3_Y2: now also J59.1 (Pin_1)
- net R3_Y3: now also J60.1 (Pin_1)
- net R3_Y4: now also J61.1 (Pin_1)
- net R3_Y5: now also J62.1 (Pin_1)
- net R3_Y6: now also J63.1 (Pin_1)
- net R3_Y7: now also J64.1 (Pin_1)
- net R4_X0: now also J33.1 (Pin_1)
- net R4_X1: now also J34.1 (Pin_1)
- net R4_X2: now also J35.1 (Pin_1)
- net R4_X3: now also J36.1 (Pin_1)
- net R4_X4: now also J37.1 (Pin_1)
- net R4_X5: now also J38.1 (Pin_1)
- net R4_X6: now also J39.1 (Pin_1)
- net R4_X7: now also J40.1 (Pin_1)
- net R4_Y0: now also J41.1 (Pin_1)
- net R4_Y1: now also J42.1 (Pin_1)
- net R4_Y2: now also J43.1 (Pin_1)
- net R4_Y3: now also J44.1 (Pin_1)
- net R4_Y4: now also J45.1 (Pin_1)
- net R4_Y5: now also J46.1 (Pin_1)
- net R4_Y6: now also J47.1 (Pin_1)
- net R4_Y7: now also J48.1 (Pin_1)
- net R5_X0: now also J17.1 (Pin_1)
- net R5_X1: now also J18.1 (Pin_1)
- net R5_X2: now also J19.1 (Pin_1)
- net R5_X3: now also J20.1 (Pin_1)
- net R5_X4: now also J21.1 (Pin_1)
- net R5_X5: now also J22.1 (Pin_1)
- net R5_X6: now also J23.1 (Pin_1)
- net R5_X7: now also J24.1 (Pin_1)
- net R5_Y0: now also J25.1 (Pin_1)
- net R5_Y1: now also J26.1 (Pin_1)
- net R5_Y2: now also J27.1 (Pin_1)
- net R5_Y3: now also J28.1 (Pin_1)
- net R5_Y4: now also J29.1 (Pin_1)
- net R5_Y5: now also J30.1 (Pin_1)
- net R5_Y6: now also J31.1 (Pin_1)
- net R5_Y7: now also J32.1 (Pin_1)
- net R7_X0: now also J1.1 (Pin_1)
- net R7_X1: now also J2.1 (Pin_1)
- net R7_X2: now also J3.1 (Pin_1)
- net R7_X3: now also J4.1 (Pin_1)
- net R7_X4: now also J5.1 (Pin_1)
- net R7_X5: now also J6.1 (Pin_1)
- net R7_X6: now also J7.1 (Pin_1)
- net R7_X7: now also J8.1 (Pin_1)
- net R7_Y0: now also J9.1 (Pin_1)
- net R7_Y1: now also J10.1 (Pin_1)
- net R7_Y2: now also J11.1 (Pin_1)
- net R7_Y3: now also J12.1 (Pin_1)
- net R7_Y4: now also J13.1 (Pin_1)
- net R7_Y5: now also J14.1 (Pin_1)
- net R7_Y6: now also J15.1 (Pin_1)
- net R7_Y7: now also J16.1 (Pin_1)
