File: KiCAD/LED_clock_logic/LED_clock_logic.kicad_sch (KiCad schematic)
At the start: 118 parts, among them J1 Socket, J10 Socket, J11 Socket, J12 Socket, J13 Socket, J14 Socket, J15 Socket, J16 Socket, J17 Socket, J18 Socket, J19 Socket, J2 Socket, J20 Socket, J21 Socket, J22 Socket, J23 Socket, J24 Socket, J25 Socket, J26 Socket, J27 Socket, J28 Socket, J29 Socket, J3 Socket, J30 Socket, J31 Socket, J32 Socket, J33 Socket, J34 Socket, J35 Socket, J36 Socket, J37 Socket, J38 Socket, J39 Socket, J4 Socket, J40 Socket, J41 Socket, J42 Socket, J43 Socket, J44 Socket, J45 Socket, J46 Socket, J47 Socket, J48 Socket, J49 Socket, J5 Socket, J50 Socket, J51 Socket, J52 Socket, J53 Socket, J54 Socket, J55 Socket, J56 Socket, J57 Socket, J58 Socket, J59 Socket, J6 Socket, J60 Socket, J61 Socket, J62 Socket, J63 Socket, J64 Socket, J65 Socket, J66 Socket, J67 Socket, J68 Socket, J69 Socket, J7 Socket, J70 Socket, J71 Socket, J72 Socket, J73 Socket, J74 Socket, J75 Socket, J76 Socket, J77 Socket, J78 Socket, J79 Socket, J8 Socket, J80 Socket, J81 Socket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

Commit message: adding Z80
Parts:
- removed U10: AVR128DB28x-xSP, Package_DIP:DIP-28_W7.62mm, symbol MCU_Microchip_AVR_Dx:AVR128DB28x-xSP
- added C11: 10uF, Capacitor_THT:CP_Radial_D5.0mm_P2.00mm, symbol Device:C
- added D1: LED, LED_THT:LED_D3.0mm, symbol Device:LED
- added D2: 1N914, Diode_THT:D_DO-15_P10.16mm_Horizontal, symbol pspice:DIODE
- added JP2: jpr3, Connector_PinSocket_2.54mm:PinSocket_1x03_P2.54mm_Vertical, symbol Device:Jumper_NC_Dual
- added R1: 470, Resistor_THT:R_Axial_DIN0207_L6.3mm_D2.5mm_P10.16mm_Horizontal, symbol Device:R_US
- added R2, R7: 4.7k, Resistor_THT:R_Axial_DIN0207_L6.3mm_D2.5mm_P10.16mm_Horizontal, symbol Device:R_US
- added R3: 1k, Resistor_THT:R_Axial_DIN0207_L6.3mm_D2.5mm_P10.16mm_Horizontal, symbol Device:R_US
- added R4: 10k, Resistor_THT:R_Axial_DIN0207_L6.3mm_D2.5mm_P10.16mm_Horizontal, symbol Device:R_US
- added SW1: SW_Push, symbol Switch:SW_Push
- added U10: 74HC14, Package_DIP:DIP-14_W7.62mm_LongPads, symbol 74xx:74HC14
- added U12: Z80CPU, Package_DIP:DIP-40_W15.24mm_Socket_LongPads, symbol CPU:Z80CPU
- added U13: AT28C256-15PU, Package_DIP:DIP-28_W15.24mm, symbol AT28C256:27256
- added U14: AS6C62256-55PCN, Package_DIP:DIP-28_W15.24mm, symbol AT28C256:27256
- added U15: 74LS32, Package_DIP:DIP-14_W7.62mm_LongPads, symbol 74xx:74LS32
- added U16, U17: 74AS74, Package_DIP:DIP-14_W7.62mm_LongPads, symbol 74xx:74LS74
- added X1: 20.000MHz, Oscillator:Oscillator_DIP-14, symbol Oscillator:ACO-xxxMHz
Connections:
- net A0: now also U12.30 (A0), U13.10 (A0), U14.10 (A0)
- net A1: now also U12.31 (A1), U13.9 (A1), U14.9 (A1)
- net A2: now also U12.32 (A2), U13.8 (A2), U14.8 (A2)
- net D0: now also U12.14 (D0), U13.11 (D0), U14.11 (D0)
- net D1: now also U12.15 (D1), U13.12 (D1), U14.12 (D1)
- net D2: now also U12.12 (D2), U13.13 (D2), U14.13 (D2)
- net D3: now also U12.8 (D3), U13.15 (D3), U14.15 (D3)
- net D4: now also U12.7 (D4), U13.16 (D4), U14.16 (D4)
- net D5: now also U12.9 (D5), U13.17 (D5), U14.17 (D5)
- net D6: now also U12.10 (D6), U13.18 (D6), U14.18 (D6)
- net D7: now also U12.13 (D7), U13.19 (D7), U14.19 (D7)
- net GND: now also U12.29 (GND), U13.14 (GND), U14.14 (GND), X1.7 (GND)
- new net: U16.3 (C), X1.8 (OUT)
- new net: D1.1 (K), U10.8
- new net: D1.2 (A), R1.1
- new net: U15.13, U17.12 (D), U17.5 (Q)
- new net: U16.12 (D), U17.9 (Q)
- new net: C11.1, D2.1 (K), R4.1, SW1.1, U10.1
- new net: C11.2, SW1.2
- new net: R7.1, U12.17 (~{NMI})
- new net: U10.9, U12.18 (~{HALT})
- new net: U10.2, U10.3
- new net: U16.2 (D), U16.6 (~{Q})
- new net: JP2.1, U15.11
- new net: U15.12, U16.8 (~{Q})
- new net +5V: D2.2 (A), JP2.3, R1.2, R2.2, R3.2, R4.2, R7.2, U12.11 (VCC), U13.28 (VCC), U14.28 (VCC), U16.1 (~{R}), U16.10 (~{S}), U16.13 (~{R}), U16.4 (~{S}), U17.1 (~{R}), U17.10 (~{S}), U17.13 (~{R}), U17.4 (~{S}), X1.14 (Vcc)
- new net A10: U12.40 (A10), U13.21 (A10), U14.21 (A10)
- new net A11: U12.1 (A11), U13.23 (A11), U14.23 (A11)
- new net A12: U12.2 (A12), U13.2 (A12), U14.2 (A12)
- new net A13: U12.3 (A13), U13.26 (A13), U14.26 (A13)
- new net A14: U12.4 (A14), U13.1 (A14), U14.1 (A14)
- new net A15: U10.5, U12.5 (A15), U15.10
- new net A3: U12.33 (A3), U13.7 (A3), U14.7 (A3)
- new net A4: U12.34 (A4), U13.6 (A4), U14.6 (A4)
- new net A5: U12.35 (A5), U13.5 (A5), U14.5 (A5)
- new net A6: U12.36 (A6), U13.4 (A6), U14.4 (A6)
- new net A7: U12.37 (A7), U13.3 (A7), U14.3 (A7)
- new net A8: U12.38 (A8), U13.25 (A8), U14.25 (A8)
- new net A9: U12.39 (A9), U13.24 (A9), U14.24 (A9)
- new net CLK: R3.1, U12.6 (~{CLK}), U16.5 (Q), U17.11 (C), U17.3 (C)
- new net nINT: R2.1, U12.16 (~{INT})
- new net nIORQ: U12.20 (~{IORQ})
- new net nM1: U12.27 (~{M1})
- new net nMRD: U13.22 (~{OE}), U14.22 (~{OE}), U15.3
- new net nMREQ: U12.19 (~{MREQ}), U15.1, U15.4, U15.9
- new net nMWR: U13.27 (nWE), U14.27 (nWE), U15.6
- new net nRAM: U10.6, U14.20 (~{CE})
- new net nRD: U12.21 (~{RD}), U15.2
- new net nROM: U13.20 (~{CE}), U15.8, U17.2 (D)
- new net nRST: U10.4, U12.26 (~{RESET})
- new net nWAIT: JP2.2, U12.24 (~{WAIT})
- new net nWR: U12.22 (~{WR}), U15.5
Other:
- note added: "2 wait states for EEPROM (need for 20MHz CPU)"
- note added: "Add 1 wait state to ROM access"
- note added: "CLOCK"
- note added: "CPU"
- note added: "EEPROM"
- note added: "May want 8, 20, 40 MHz options"
- note added: "Memory strobes"
- note added: "RAM"
- note added: "RESET"
- note added: "ROM WAIT STATES"
- moved on the sheet: J1, J10, J11, J12, J13, J14, J15, J16, J17, J18, J19, J2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

Commit message: tentative placement
Other:
- moved on the sheet: D1, R1, R2, R7, U10D, U11, U12, U13, U14
