File: KiCAD/LED_clock_only1/LED_clock_only1.kicad_sch (KiCad schematic)
At the start: 392 parts, among them J1 CONN_2X10, U1 ICM7218A, U2 ICM7218A, U3 ICM7218A, U4 ICM7218A, U5 ICM7218A, U6 ICM7218A, U7 74HC138, U8 74LS244, U9 74LS125

Commit message: tentative placement
Parts:
- C1, C2, C3, C4, C5, C6, C7, C8, C9: footprint Capacitor_SMD:C_1206_3216Metric_Pad1.33x1.80mm_HandSolder -> Capacitor_THT:C_Disc_D4.3mm_W1.9mm_P5.00mm
- U1, U2, U3, U4, U5, U6: footprint Package_LCC:PLCC-28 -> Package_DIP:DIP-28_W15.24mm_LongPads
- U7: footprint Package_SO:SO-16_3.9x9.9mm_P1.27mm -> Package_DIP:DIP-16_W7.62mm_LongPads; DigiKey MM74HC138M-ND -> (none)
- U8: footprint Package_SO:SO-20_5.3x12.6mm_P1.27mm -> Package_DIP:DIP-20_W7.62mm_LongPads; DigiKey 296-8274-1-ND -> (none)
- U9: footprint Package_SO:SO-14_3.9x8.65mm_P1.27mm -> Package_DIP:DIP-14_W7.62mm_LongPads; DigiKey MC74HC125ADR2GOSCT-ND -> (none)
Changed lines of the file:
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@@
 			)
 		)
-		(property "Footprint" "Package_LCC:PLCC-28"
+		(property "Footprint" "Package_DIP:DIP-28_W15.24mm_LongPads"
 			(at 185.42 166.37 0)
 			(effects
@@
 			)
 		)
-		(property "Footprint" "Package_LCC:PLCC-28"
+		(property "Footprint" "Package_DIP:DIP-28_W15.24mm_LongPads"
 			(at 351.79 165.1 0)
 			(effects
@@
 		(on_board yes)
 		(dnp no)
+		(fields_autoplaced yes)
 		(property "Reference" "U7"
 			(at 102.4733 175.26 0)
@@
 			)
 		)
-		(property "Footprint" "Package_SO:SO-16_3.9x9.9mm_P1.27mm"
+		(property "Footprint" "Package_DIP:DIP-16_W7.62mm_LongPads"
 			(at 100.33 193.04 0)
 			(effects
@@
 			)
 		)
-		(property "DigiKey" "MM74HC138M-ND"
-			(at 114.808 204.724 0)
-			(effects
-				(font
-					(size 1.27 1.27)
-				)
-			)
-		)
 		(pin "10"
 		)
@@
 			)
 		)
-		(property "Footprint" "Capacitor_SMD:C_1206_3216Metric_Pad1.33x1.80mm_HandSolder"
+		(property "Footprint" "Capacitor_THT:C_Disc_D4.3mm_W1.9mm_P5.00mm"
 			(at 214.3252 250.19 0)
 			(effects
@@
 			)
 		)
-		(property "Footprint" "Package_SO:SO-14_3.9x8.65mm_P1.27mm"
+		(property "Footprint" "Package_DIP:DIP-14_W7.62mm_LongPads"
 			(at 151.13 245.11 0)
 			(effects
@@
 			)
 		)
-		(property "DigiKey" "MC74HC125ADR2GOSCT-ND"
-			(at 165.608 254.762 0)
-			(effects
-				(font
-					(size 1.27 1.27)
-				)
-			)
-		)
 		(pin "3"
 		)
@@
 			)
 		)
-		(property "Footprint" "Package_SO:SO-14_3.9x8.65mm_P1.27mm"
+		(property "Footprint" "Package_DIP:DIP-14_W7.62mm_LongPads"
 			(at 60.96 208.28 0)
 			(effects
@@
 			)
 		)
-		(property "DigiKey" "MC74HC125ADR2GOSCT-ND"
-			(at 60.96 208.28 0)
-			(effects
-				(font
-					(size 1.27 1.27)
-				)
-				(hide yes)
-			)
-		)
 		(pin "3"
 		)
@@
 		(on_board yes)
 		(dnp no)
+		(fields_autoplaced yes)
 		(property "Reference" "U8"
 			(at 102.4733 215.9 0)
@@
 			)
 		)
-		(property "Footprint" "Package_SO:SO-20_5.3x12.6mm_P1.27mm"
+		(property "Footprint" "Package_DIP:DIP-20_W7.62mm_LongPads"
 			(at 100.33 236.22 0)
 			(effects
@@
 			)
 		)
-		(property "DigiKey" "296-8274-1-ND"
-			(at 111.506 253.746 0)
-			(effects
-				(font
-					(size 1.27 1.27)
-				)
-			)
-		)
 		(pin "10"
 		)
@@
 			)
 		)
-		(property "Footprint" "Capacitor_SMD:C_1206_3216Metric_Pad1.33x1.80mm_HandSolder"
+		(property "Footprint" "Capacitor_THT:C_Disc_D4.3mm_W1.9mm_P5.00mm"
 			(at 227.0252 250.19 0)
 			(effects
@@
 			)
 		)
-		(property "Footprint" "Package_LCC:PLCC-28"
+		(property "Footprint" "Package_DIP:DIP-28_W15.24mm_LongPads"
 			(at 308.61 166.37 0)
 			(effects
@@
 			)
 		)
-		(property "Footprint" "Capacitor_SMD:C_1206_3216Metric_Pad1.33x1.80mm_HandSolder"
+		(property "Footprint" "Capacitor_THT:C_Disc_D4.3mm_W1.9mm_P5.00mm"
 			(at 201.6252 250.19 0)
 			(effects
@@
 			)
 		)
-		(property "Footprint" "Capacitor_SMD:C_1206_3216Metric_Pad1.33x1.80mm_HandSolder"
+		(property "Footprint" "Capacitor_THT:C_Disc_D4.3mm_W1.9mm_P5.00mm"
 			(at 188.9252 250.19 0)
 			(effects
@@
 			)
 		)
-		(property "Footprint" "Package_LCC:PLCC-28"
+		(property "Footprint" "Package_DIP:DIP-28_W15.24mm_LongPads"
 			(at 398.78 165.1 0)
 			(effects
@@
 			)
 		)
-		(property "Footprint" "Package_LCC:PLCC-28"
+		(property "Footprint" "Package_DIP:DIP-28_W15.24mm_LongPads"
 			(at 226.06 165.1 0)
 			(effects
@@
 			)
 		)
-		(property "Footprint" "Package_LCC:PLCC-28"
+		(property "Footprint" "Package_DIP:DIP-28_W15.24mm_LongPads"
 			(at 266.7 166.37 0)
 			(effects
@@
 			)
 		)
-		(property "Footprint" "Capacitor_SMD:C_1206_3216Metric_Pad1.33x1.80mm_HandSolder"
+		(property "Footprint" "Capacitor_THT:C_Disc_D4.3mm_W1.9mm_P5.00mm"
 			(at 207.9752 250.19 0)
 			(effects
@@
 			)
 		)
-		(property "Footprint" "Capacitor_SMD:C_1206_3216Metric_Pad1.33x1.80mm_HandSolder"
+		(property "Footprint" "Capacitor_THT:C_Disc_D4.3mm_W1.9mm_P5.00mm"
 			(at 220.6752 250.19 0)
 			(effects
@@
 			)
 		)
-		(property "Footprint" "Capacitor_SMD:C_1206_3216Metric_Pad1.33x1.80mm_HandSolder"
+		(property "Footprint" "Capacitor_THT:C_Disc_D4.3mm_W1.9mm_P5.00mm"
 			(at 233.3752 250.19 0)
 			(effects
@@
 			)
 		)
-		(property "Footprint" "Capacitor_SMD:C_1206_3216Metric_Pad1.33x1.80mm_HandSolder"
+		(property "Footprint" "Capacitor_THT:C_Disc_D4.3mm_W1.9mm_P5.00mm"
 			(at 195.2752 250.19 0)
 			(effects
@@
 			)
 		)
-		(property "Footprint" "Capacitor_SMD:C_1206_3216Metric_Pad1.33x1.80mm_HandSolder"
+		(property "Footprint" "Capacitor_THT:C_Disc_D4.3mm_W1.9mm_P5.00mm"
 			(at 239.7252 250.19 0)
 			(effects
