File: KiCAD/LED_proto_sector/LED_proto_sector.kicad_pcb (KiCad board)
At the start: 2 copper layers, 114.3 x 120.7 mm, 70 parts, among them J2 PJ-082BH, U1 ICM7218A

Commit message: prototype sector
Parts:
- added A1: Arduino_UNO_R3, Module:Arduino_UNO_R3, B.Cu at (191.8, 105.4)
- added JP1: Jumper_2_Open, Connector_PinHeader_2.54mm:PinHeader_1x02_P2.54mm_Vertical, F.Cu at (156.2, 116.8)
- C1: moved to B.Cu
- moved H1 189.3 mm to (229.9, 109.9)
- moved H3 183.9 mm to (229.9, 157.5)
- moved H2 176.6 mm to (229.9, 62.2)
- moved H4 118.9 mm to (143.5, 157.5)
- moved H5 105.1 mm to (143.5, 62.2)
- moved D70 52.8 mm to (221.0, 97.8)
- moved D10 51.4 mm to (219.7, 62.2)
- moved C1 51.0 mm to (193.7, 120.4), turned to 0 degrees
- moved D69 47.1 mm to (213.4, 97.8)
- moved D60 46.0 mm to (221.0, 92.7)
- moved D9 43.7 mm to (212.1, 62.2)
- moved D68 41.9 mm to (205.7, 97.8)
- moved D50 40.9 mm to (221.0, 87.6)
- moved D30 40.2 mm to (221.0, 77.5)
- moved D59 40.0 mm to (213.4, 92.7)
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Routing:
- net /Sector1/LD7: track 0.00 -> 177.7 mm, vias 0 -> 1
- net /Sector1/Sb: track 0.00 -> 170.0 mm, vias 0 -> 1
- net /Sector1/Sc: track 0.00 -> 159.7 mm
- net /Sector1/Se: track 0.00 -> 153.6 mm, vias 0 -> 6
- net /Sector1/Sa: track 0.00 -> 144.0 mm, vias 0 -> 3
- net /Sector1/Sd: track 0.00 -> 130.4 mm, vias 0 -> 5
- net /Sector1/LD1: track 0.00 -> 118.9 mm
- net /Sector1/dp: track 0.00 -> 112.5 mm, vias 0 -> 4
- net /Sector1/LD3: track 0.00 -> 107.9 mm, vias 0 -> 10
- net /Sector1/LD2: track 0.00 -> 107.4 mm, vias 0 -> 8
- net /Sector1/Sf: track 0.00 -> 105.7 mm, vias 0 -> 3
- net /Sector1/LD4: track 0.00 -> 99.1 mm, vias 0 -> 10
- net /Sector1/LD5: track 0.00 -> 91.6 mm, vias 0 -> 8
- net /Sector1/Sg: track 0.00 -> 91.1 mm, vias 0 -> 4
- net /Sector1/LD6: track 0.00 -> 84.8 mm, vias 0 -> 8
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- added copper zone on F.Cu, net +5V
- added copper zone on B.Cu, net GND
Other:
- board size 114.3 x 120.7 mm -> 96.5 x 108 mm
- board text added: "CLOCK V0.1 ESH 2026-01"
- board text removed: "CLOCK V1.0 ESH 2026-01"
