File: KiCAD/Led_clock_sector/Led_clock_sector.kicad_sch (KiCad schematic)
At the start: 0 parts

Commit message: Sector-based layout
Other:
- note added: "Sectors 1-6 organized clockwise, with sector 1 handling 12:00-1:59"
- note added: "UPCO LED Clock"

Commit message: rev 1?
Parts:
- added A1: Arduino_Nano_ESP32, Module:Arduino_Nano, symbol MCU_Module:Arduino_Nano_ESP32
- added C10, C7, C8, C9: 0.1uF, Capacitor_SMD:C_1206_3216Metric_Pad1.33x1.80mm_HandSolder, symbol Device:C
- added H1, H2, H3, H4, H5: MountingHole, MountingHole:MountingHole_4.3mm_M4, symbol Mechanical:MountingHole
- added J1: Conn_01x04, Connector_PinHeader_2.54mm:PinHeader_1x04_P2.54mm_Vertical, symbol Connector_Generic:Conn_01x04
- added J2: PJ-082BH, my_BJack:SAMESKY_PJ-082BH, symbol PJ-082BH:PJ-082BH
- added U2, U3: SN74LVC4245ADWR, my_TI_24N:SOIC127P1030X265-24N, symbol SN74LVC4245ADWR:SN74LVC4245ADWR
Connections:
- net D0: now also U2.3 (A1)
- net D1: now also U2.4 (A2)
- net D2: now also U2.5 (A3)
- net D3: now also U2.6 (A4)
- net D4: now also U2.7 (A5)
- net D5: now also U2.8 (A6)
- net D6: now also U2.9 (A7)
- net D7: now also U2.10 (A8)
- net MODE: now also U3.9 (A7)
- net ~{WR0}: now also U3.3 (A1)
- net ~{WR1}: now also U3.4 (A2)
- net ~{WR2}: now also U3.5 (A3)
- net ~{WR3}: now also U3.6 (A4)
- net ~{WR4}: now also U3.7 (A5)
- net ~{WR5}: now also U3.8 (A6)
- new net: A1.2 (D0/RX), J1.2 (Pin_2)
- new net: A1.1 (D1/TX), J1.3 (Pin_3)
- new net +3.3V: A1.17 (3V3), C10.1, C7.1, U2.23 (VCCB_(3.3_V)), U2.24 (VCCB_(3.3_V)_2), U3.23 (VCCB_(3.3_V)), U3.24 (VCCB_(3.3_V)_2)
- new net +5V: A1.30 (VIN), C8.1, C9.1, J1.1 (Pin_1), J2.1, U2.1 ((5_V)_VCCA), U3.1 ((5_V)_VCCA)
- new net ED0: A1.19 (A0), U2.21 (B1)
- new net ED1: A1.20 (A1), U2.20 (B2)
- new net ED2: A1.21 (A2), U2.19 (B3)
- new net ED3: A1.22 (A3), U2.18 (B4)
- new net ED4: A1.23 (SDA/A4), U2.17 (B5)
- new net ED5: A1.24 (SCL/A5), U2.16 (B6)
- new net ED6: A1.25 (A6), U2.15 (B7)
- new net ED7: A1.26 (A7), U2.14 (B8)
- new net EMODE: A1.11 (D8), U3.15 (B7)
- new net GND: A1.29 (GND), A1.4 (GND), C10.2, C7.2, C8.2, C9.2, J1.4 (Pin_4), J2.2, J2.SH1 (SHIELD), J2.SH2 (SHIELD__1), J2.SH3 (SHIELD__2), J2.SH4 (SHIELD__3), U2.11 (GND), U2.12 (GND__1), U2.13 (GND__2), U2.2 (DIR), U2.22 (~{OE}), U3.11 (GND), U3.12 (GND__1), U3.13 (GND__2), U3.2 (DIR), U3.22 (~{OE})
- new net ~{EWR0}: A1.5 (D2), U3.21 (B1)
- new net ~{EWR1}: A1.6 (D3), U3.20 (B2)
- new net ~{EWR2}: A1.7 (D4), U3.19 (B3)
- new net ~{EWR3}: A1.8 (D5), U3.18 (B4)
- new net ~{EWR4}: A1.9 (D6), U3.17 (B5)
- new net ~{EWR5}: A1.10 (D7), U3.16 (B6)

Commit message: update
Parts:
- added N1: Socket DIP-32, symbol Mechanical:Housing
- A1: CatNo (none) -> 1050-ABX00083-ND
- C10, C7, C8, C9: CatNo (none) -> 4713-GMC31X7R104K10NTCT-ND
- H1, H2, H3, H4, H5, J1: CatNo (none) -> N/A
- J2: CatNo (none) -> CP-082BHCT-ND
- U2, U3: CatNo (none) -> 296-14911-1-ND
Changed lines of the file:
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@@
+			)
+		)
+		(property "CatNo" "4713-GMC31X7R104K10NTCT-ND"
+			(at 182.626 125.73 90)
+			(effects
+				(font
+					(size 1.27 1.27)
+				)
 			)
 		)
@@
 			)
 		)
+		(property "CatNo" "N/A"
+			(at 91.44 168.91 0)
+			(effects
+				(font
+					(size 1.27 1.27)
+				)
+				(hide yes)
+			)
+		)
 		(instances
 			(project ""
@@
 		(on_board yes)
 		(dnp no)
-		(fields_autoplaced yes)
 		(property "Reference" "J2"
 			(at 44.45 36.83 0)
@@
 				(justify bottom)
 				(hide yes)
+			)
+		)
+		(property "CatNo" "CP-082BHCT-ND"
+			(at 44.196 67.818 0)
+			(effects
+				(font
+					(size 1.27 1.27)
+				)
 			)
 		)
@@
 			)
 		)
+		(property "CatNo" "4713-GMC31X7R104K10NTCT-ND"
+			(at 273.05 101.6 0)
+			(effects
+				(font
+					(size 1.27 1.27)
+				)
+				(hide yes)
+			)
+		)
 		(pin "1"
 		)
@@
 		(on_board yes)
 		(dnp no)
-		(fields_autoplaced yes)
 		(property "Reference" "U2"
 			(at 149.86 86.36 0)
@@
 				)
 				(hide yes)
+			)
+		)
+		(property "CatNo" "296-14911-1-ND"
+			(at 150.622 149.606 0)
+			(effects
+				(font
+					(size 1.27 1.27)
+				)
 			)
 		)
@@
 			)
 		)
+		(property "CatNo" "296-14911-1-ND"
+			(at 236.22 115.57 0)
+			(effects
+				(font
+					(size 1.27 1.27)
+				)
+				(hide yes)
+			)
+		)
 		(pin "13"
 		)
@@
 			)
 		)
+		(property "CatNo" "N/A"
+			(at 27.94 113.03 0)
+			(effects
+				(font
+					(size 1.27 1.27)
+				)
+				(hide yes)
+			)
+		)
 		(pin "2"
 		)
@@
 			)
 		)
+		(property "CatNo" "N/A"
+			(at 91.44 179.07 0)
+			(effects
+				(font
+					(size 1.27 1.27)
+				)
+				(hide yes)
+			)
+		)
 		(instances
 			(project "Led_clock_sector"
@@
 			)
 		)
+		(property "CatNo" "N/A"
+			(at 91.44 189.23 0)
+			(effects
+				(font
+					(size 1.27 1.27)
+				)
+				(hide yes)
+			)
+		)
 		(instances
 			(project "Led_clock_sector"
 				(path "/854da954-ecec-4a18-8053-33c879b37ebb"
 					(reference "H5")
+					(unit 1)
+				)
+			)
+		)
+	)
+	(symbol
+		(lib_id "Mechanical:Housing")
+		(at 31.75 168.91 0)
+		(unit 1)
+		(exclude_from_sim no)
+		(in_bom yes)
+		(on_board yes)
+		(dnp no)
+		(property "Reference" "N1"
+			(at 35.56 167.9574 0)
+			(effects
+				(font
+					(size 1.27 1.27)
+				)
+				(justify left)
+			)
+		)
+		(property "Value" "Socket DIP-32"
+			(at 35.56 170.4974 0)
+			(effects
+				(font
+					(size 1.27 1.27)
+				)
+				(justify left)
+			)
+		)
+		(property "Footprint" ""
+			(at 33.02 167.64 0)
+			(effects
+				(font
+					(size 1.27 1.27)
+				)
+				(hide yes)
+			)
+		)
+		(property "Datasheet" "~"
+			(at 33.02 167.64 0)
+			(effects
+				(font
+					(size 1.27 1.27)
+				)
+				(hide yes)
+			)
+		)
+		(property "Description" "Housing"
+			(at 31.75 168.91 0)
+			(effects
+				(font
+					(size 1.27 1.27)
+				)
+				(hide yes)
+			)
+		)
+		(property "CatNo" "A120356-ND"
+			(at 41.656 173.228 0)
+			(effects
+				(font
+					(size 1.27 1.27)
+				)
+			)
+		)
+		(instances
+			(project ""
+				(path "/854da954-ecec-4a18-8053-33c879b37ebb"
+					(reference "N1")
 					(unit 1)
 				)
@@
 			)
 		)
+		(property "CatNo" "N/A"
+			(at 91.44 173.99 0)
+			(effects
+				(font
+					(size 1.27 1.27)
+				)
+				(hide yes)
+			)
+		)
 		(instances
 			(project "Led_clock_sector"
@@
 			)
 		)
+		(property "CatNo" "N/A"
+			(at 91.44 184.15 0)
+			(effects
+				(font
+					(size 1.27 1.27)
+				)
+				(hide yes)
+			)
+		)
 		(instances
 			(project "Led_clock_sector"
@@
 		(on_board yes)
 		(dnp no)
-		(fields_autoplaced yes)
 		(property "Reference" "A1"
 			(at 64.77 100.33 0)
@@
 				)
 				(hide yes)
+			)
+		)
+		(property "CatNo" "1050-ABX00083-ND"
+			(at 77.216 153.416 0)
+			(effects
+				(font
+					(size 1.27 1.27)
+				)
 			)
 		)
@@
 			)
 		)
+		(property "CatNo" "4713-GMC31X7R104K10NTCT-ND"
+			(at 187.96 102.87 0)
+			(effects
+				(font
+					(size 1.27 1.27)
+				)
+				(hide yes)
+			)
+		)
 		(pin "1"
 		)
@@
 			(at 266.7 101.6 0)
 			(effects
+				(font
+					(size 1.27 1.27)
+				)
+				(hide yes)
+			)
+		)
+		(property "CatNo" "4713-GMC31X7R104K10NTCT-ND"
+			(at 266.7 101.6 0)
+			(effects
