File: KiCAD/Led_clock_sector/sector.kicad_sch (KiCad schematic)
At the start: 63 parts, among them U1 ICM7218A

Commit message: Sector-based layout
Parts:
- D1: renamed from D; footprint (none) -> LED_THT:LED_D3.0mm
- D10, D2, D3, D4, D5, D6, D7, D8, D9: footprint (none) -> LED_THT:LED_D3.0mm
- D11, D12: footprint (none) -> LED_THT:LED_D5.0mm
- D21, D22, D23, D24, D25, D26, D27, D28, D29, D30, D31, D32, D33, D34, D35, D36, D37, D38, D39, D40, D41, D42, D43, D44, D45, D46, D47, D48, D49, D50, D51, D52, D53, D54, D55, D56, D57, D58, D59, D60, D61, D62, D63, D64, D65, D66, D67, D68, D69, D70: footprint (none) -> LED_SMD:LED_1206_3216Metric_Pad1.42x1.75mm_HandSolder
Connections:
- net D1: no longer D1.2 (A), D2.2 (A), D3.2 (A), D4.2 (A), D5.2 (A), D6.2 (A), D7.2 (A), D8.2 (A), U1.15 (d1)
- net D2: no longer D21.2 (A), D22.2 (A), D23.2 (A), D24.2 (A), D25.2 (A), D26.2 (A), D27.2 (A), D28.2 (A), U1.16 (d2)
- net D3: no longer D31.2 (A), D32.2 (A), D33.2 (A), D34.2 (A), D35.2 (A), D36.2 (A), D37.2 (A), D38.2 (A), U1.23 (d3)
- net D4: no longer D41.2 (A), D42.2 (A), D43.2 (A), D44.2 (A), D45.2 (A), D46.2 (A), D47.2 (A), D48.2 (A), U1.20 (d4)
- net D5: no longer D51.2 (A), D52.2 (A), D53.2 (A), D54.2 (A), D55.2 (A), D56.2 (A), D57.2 (A), D58.2 (A), U1.17 (d5)
- net D6: no longer D61.2 (A), D62.2 (A), D63.2 (A), D64.2 (A), D65.2 (A), D66.2 (A), D67.2 (A), D68.2 (A), U1.22 (d6)
- net D7: no longer D10.2 (A), D11.2 (A), D12.2 (A), D29.2 (A), D30.2 (A), D39.2 (A), D40.2 (A), D9.2 (A), U1.21 (d7)
- net D8 renamed LD8
- new net LD1: D1.2 (A), D2.2 (A), D3.2 (A), D4.2 (A), D5.2 (A), D6.2 (A), D7.2 (A), D8.2 (A), U1.15 (d1)
- new net LD2: D21.2 (A), D22.2 (A), D23.2 (A), D24.2 (A), D25.2 (A), D26.2 (A), D27.2 (A), D28.2 (A), U1.16 (d2)
- new net LD3: D31.2 (A), D32.2 (A), D33.2 (A), D34.2 (A), D35.2 (A), D36.2 (A), D37.2 (A), D38.2 (A), U1.23 (d3)
- new net LD4: D41.2 (A), D42.2 (A), D43.2 (A), D44.2 (A), D45.2 (A), D46.2 (A), D47.2 (A), D48.2 (A), U1.20 (d4)
- new net LD5: D51.2 (A), D52.2 (A), D53.2 (A), D54.2 (A), D55.2 (A), D56.2 (A), D57.2 (A), D58.2 (A), U1.17 (d5)
- new net LD6: D61.2 (A), D62.2 (A), D63.2 (A), D64.2 (A), D65.2 (A), D66.2 (A), D67.2 (A), D68.2 (A), U1.22 (d6)
- new net LD7: D10.2 (A), D11.2 (A), D12.2 (A), D29.2 (A), D30.2 (A), D39.2 (A), D40.2 (A), D9.2 (A), U1.21 (d7)
Other:
- note added: "Ring 1 - 3mm"
- note added: "Ring 2 - 5mm"
- note added: "Ring 3 - 1206"
- note added: "Ring 4 - 1206"
- note added: "Ring 5 - 1206"
- note added: "Ring 6 - 1206"
- note added: "Ring 7 - 1206"
- moved on the sheet: D1, D10, D11, D12, D2, D21, D22, D23, D24, D25, D26, D27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

Commit message: rev 1?
Parts:
- added C1: 0.1uF, Capacitor_SMD:C_1206_3216Metric_Pad1.33x1.80mm_HandSolder, symbol Device:C
- U1: DigiKey (none) -> ICM7218AIQI+-ND
Connections:
- net GND: now also C1.2
- net VCC renamed +5V
- net +5V: now also C1.1
Changed lines of the file:
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@@
 	)
 	(junction
+		(at 45.72 22.86)
+		(diameter 0)
+		(color 0 0 0 0)
+	)
+	(junction
 		(at 127 120.65)
 		(diameter 0)
@@
 	(wire
 		(pts
+			(xy 53.34 22.86) (xy 45.72 22.86)
+		)
+		(stroke
+			(width 0)
+			(type default)
+		)
+	)
+	(wire
+		(pts
 			(xy 101.6 120.65) (xy 101.6 135.89)
 		)
@@
 	(wire
 		(pts
-			(xy 45.72 33.02) (xy 45.72 38.1)
+			(xy 45.72 22.86) (xy 45.72 38.1)
 		)
 		(stroke
@@
 			)
 		)
+		(property "DigiKey" "ICM7218AIQI+-ND"
+			(at 56.134 36.83 0)
+			(effects
+				(font
+					(size 1.27 1.27)
+				)
+			)
+		)
 		(pin "22"
 		)
@@
 	)
 	(symbol
-		(lib_id "power:VCC")
-		(at 45.72 33.02 0)
-		(unit 1)
-		(exclude_from_sim no)
-		(in_bom yes)
-		(on_board yes)
-		(dnp no)
-		(fields_autoplaced yes)
-		(property "Reference" "#PWR0101"
-			(at 45.72 36.83 0)
-			(effects
-				(font
-					(size 1.27 1.27)
-				)
-				(hide yes)
-			)
-		)
-		(property "Value" "VCC"
-			(at 45.72 27.94 0)
-			(effects
-				(font
-					(size 1.27 1.27)
-				)
-			)
-		)
-		(property "Footprint" ""
-			(at 45.72 33.02 0)
-			(effects
-				(font
-					(size 1.27 1.27)
-				)
-				(hide yes)
-			)
-		)
-		(property "Datasheet" ""
-			(at 45.72 33.02 0)
-			(effects
-				(font
-					(size 1.27 1.27)
-				)
-				(hide yes)
-			)
-		)
-		(property "Description" "Power symbol creates a global label with name \"VCC\""
-			(at 45.72 33.02 0)
-			(effects
-				(font
-					(size 1.27 1.27)
-				)
-				(hide yes)
-			)
-		)
-		(pin "1"
-		)
-		(instances
-			(project "Led_clock_sector"
-				(path "/854da954-ecec-4a18-8053-33c879b37ebb/04b05e74-e8a7-427c-8af0-1f08c509c03f"
-					(reference "#PWR057")
-					(unit 1)
-				)
-				(path "/854da954-ecec-4a18-8053-33c879b37ebb/1f856a04-686b-457e-87a4-7af76d5edd09"
-					(reference "#PWR053")
-					(unit 1)
-				)
-				(path "/854da954-ecec-4a18-8053-33c879b37ebb/5d46d765-1d6c-4220-8ee8-442dc3b3697f"
-					(reference "#PWR055")
-					(unit 1)
-				)
-				(path "/854da954-ecec-4a18-8053-33c879b37ebb/929ff51f-02c5-4c2a-9e52-da6367ed83c7"
-					(reference "#PWR0101")
-					(unit 1)
-				)
-				(path "/854da954-ecec-4a18-8053-33c879b37ebb/9a15f943-25f9-4164-acd0-5bc298e32013"
-					(reference "#PWR061")
-					(unit 1)
-				)
-				(path "/854da954-ecec-4a18-8053-33c879b37ebb/ab90faec-1c29-4b43-b677-784af5a0f47e"
-					(reference "#PWR059")
-					(unit 1)
-				)
-			)
-		)
-	)
-	(symbol
 		(lib_id "Device:LED")
 		(at 129.54 82.55 270)
@@
 	)
 	(symbol
+		(lib_id "power:+5V")
+		(at 45.72 22.86 0)
+		(unit 1)
+		(exclude_from_sim no)
+		(in_bom yes)
+		(on_board yes)
+		(dnp no)
+		(fields_autoplaced yes)
+		(property "Reference" "#PWR01"
+			(at 45.72 26.67 0)
+			(effects
+				(font
+					(size 1.27 1.27)
+				)
+				(hide yes)
+			)
+		)
+		(property "Value" "+5V"
+			(at 45.72 17.78 0)
+			(effects
+				(font
+					(size 1.27 1.27)
+				)
+			)
+		)
+		(property "Footprint" ""
+			(at 45.72 22.86 0)
+			(effects
+				(font
+					(size 1.27 1.27)
+				)
+				(hide yes)
+			)
+		)
+		(property "Datasheet" ""
+			(at 45.72 22.86 0)
+			(effects
+				(font
+					(size 1.27 1.27)
+				)
+				(hide yes)
+			)
+		)
+		(property "Description" "Power symbol creates a global label with name \"+5V\""
+			(at 45.72 22.86 0)
+			(effects
+				(font
+					(size 1.27 1.27)
+				)
+				(hide yes)
+			)
+		)
+		(pin "1"
+		)
+		(instances
+			(project ""
+				(path "/854da954-ecec-4a18-8053-33c879b37ebb/04b05e74-e8a7-427c-8af0-1f08c509c03f"
+					(reference "#PWR04")
+					(unit 1)
+				)
+				(path "/854da954-ecec-4a18-8053-33c879b37ebb/1f856a04-686b-457e-87a4-7af76d5edd09"
+					(reference "#PWR02")
+					(unit 1)
+				)
+				(path "/854da954-ecec-4a18-8053-33c879b37ebb/5d46d765-1d6c-4220-8ee8-442dc3b3697f"
+					(reference "#PWR03")
+					(unit 1)
+				)
+				(path "/854da954-ecec-4a18-8053-33c879b37ebb/929ff51f-02c5-4c2a-9e52-da6367ed83c7"
+					(reference "#PWR01")
+					(unit 1)
+				)
+				(path "/854da954-ecec-4a18-8053-33c879b37ebb/9a15f943-25f9-4164-acd0-5bc298e32013"
+					(reference "#PWR06")
+					(unit 1)
+				)
+				(path "/854da954-ecec-4a18-8053-33c879b37ebb/ab90faec-1c29-4b43-b677-784af5a0f47e"
+					(reference "#PWR05")
+					(unit 1)
+				)
+			)
+		)
+	)
+	(symbol
 		(lib_id "Device:LED")
 		(at 78.74 82.55 270)
@@
 	)
 	(symbol
+		(lib_id "Device:C")
+		(at 53.34 26.67 0)
+		(unit 1)
+		(exclude_from_sim no)
+		(in_bom yes)
+		(on_board yes)
+		(dnp no)
+		(fields_autoplaced yes)
+		(property "Reference" "C1"
+			(at 57.15 25.3999 0)
+			(effects
+				(font
+					(size 1.27 1.27)
+				)
+				(justify left)
+			)
+		)
+		(property "Value" "0.1uF"
+			(at 57.15 27.9399 0)
+			(effects
+				(font
+					(size 1.27 1.27)
+				)
+				(justify left)
+			)
+		)
+		(property "Footprint" "Capacitor_SMD:C_1206_3216Metric_Pad1.33x1.80mm_HandSolder"
+			(at 54.3052 30.48 0)
+			(effects
+				(font
+					(size 1.27 1.27)
+				)
+				(hide yes)
+			)
+		)
+		(property "Datasheet" "~"
+			(at 53.34 26.67 0)
+			(effects
+				(font
+					(size 1.27 1.27)
+				)
+				(hide yes)
+			)
+		)
+		(property "Description" "Unpolarized capacitor"
+			(at 53.34 26.67 0)
+			(effects
+				(font
+					(size 1.27 1.27)
+				)
+				(hide yes)
+			)
+		)
+		(pin "1"
+		)
+		(pin "2"
+		)
+		(instances
+			(project ""
+				(path "/854da954-ecec-4a18-8053-33c879b37ebb/04b05e74-e8a7-427c-8af0-1f08c509c03f"
+					(reference "C4")
+					(unit 1)
+				)
+				(path "/854da954-ecec-4a18-8053-33c879b37ebb/1f856a04-686b-457e-87a4-7af76d5edd09"
+					(reference "C2")
+					(unit 1)
+				)
+				(path "/854da954-ecec-4a18-8053-33c879b37ebb/5d46d765-1d6c-4220-8ee8-442dc3b3697f"
+					(reference "C3")
+					(unit 1)
+				)
+				(path "/854da954-ecec-4a18-8053-33c879b37ebb/929ff51f-02c5-4c2a-9e52-da6367ed83c7"
+					(reference "C1")
+					(unit 1)
+				)
+				(path "/854da954-ecec-4a18-8053-33c879b37ebb/9a15f943-25f9-4164-acd0-5bc298e32013"
+					(reference "C6")
+					(unit 1)
+				)
+				(path "/854da954-ecec-4a18-8053-33c879b37ebb/ab90faec-1c29-4b43-b677-784af5a0f47e"
+					(reference "C5")
+					(unit 1)
+				)
+			)
+		)
+	)
+	(symbol
 		(lib_id "Device:LED")
 		(at 97.79 110.49 270)
@@
 					(unit 1)
 				)
+			)
+		)
+	)
+	(symbol
+		(lib_id "power:GND")
+		(at 53.34 30.48 0)
+		(unit 1)
+		(exclude_from_sim no)
+		(in_bom yes)
+		(on_board yes)
+		(dnp no)
+		(property "Reference" "#PWR07"
+			(at 53.34 36.83 0)
+			(effects
+				(font
+					(size 1.27 1.27)
+				)
+				(hide yes)
+			)
+		)
+		(property "Value" "GND"
+			(at 57.404 32.766 0)
+			(effects
+				(font
+					(size 1.27 1.27)
+				)
+			)
+		)
+		(property "Footprint" ""
+			(at 53.34 30.48 0)
+			(effects
+				(font
+					(size 1.27 1.27)
+				)
+				(hide yes)
+			)
+		)
+		(property "Datasheet" ""
+			(at 53.34 30.48 0)
+			(effects
+				(font
+					(size 1.27 1.27)
+				)
+				(hide yes)
+			)
+		)
+		(property "Description" "Power symbol creates a global label with name \"GND\" , ground"
+			(at 53.34 30.48 0)
+			(effects
+				(font
+					(size 1.27 1.27)
+				)
+				(hide yes)
+			)
+		)
+		(pin "1"
+		)
+		(instances
+			(project "Led_clock_sector"
+				(path "/854da954-ecec-4a18-8053-33c879b37ebb/04b05e74-e8a7-427c-8af0-1f08c509c03f"
+					(reference "#PWR010")
+					(unit 1)
+				)
+				(path "/854da954-ecec-4a18-8053-33c879b37ebb/1f856a04-686b-457e-87a4-7af76d5edd09"
+					(reference "#PWR08")
+					(unit 1)
+				)
+				(path "/854da954-ecec-4a18-8053-33c879b37ebb/5d46d765-1d6c-4220-8ee8-442dc3b3697f"
+					(reference "#PWR09")
+					(unit 1)
+				)
+				(path "/854da954-ecec-4a18-8053-33c879b37ebb/929ff51f-02c5-4c2a-9e52-da6367ed83c7"
+					(reference "#PWR07")
+					(unit 1)
+				)
+				(path "/854da954-ecec-4a18-8053-33c879b37ebb/9a15f943-25f9-4164-acd0-5bc298e32013"
+					(reference "#PWR012")
+					(unit 1)
+				)
+				(path "/854da954-ecec-4a18-8053-33c879b37ebb/ab90faec-1c29-4b43-b677-784af5a0f47e"
+					(reference "#PWR011")
+					(unit 1)
+				)

Commit message: update
Parts:
- C1: CatNo (none) -> 4713-GMC31X7R104K10NTCT-ND
- D1, D10, D2, D3, D4, D5, D6, D7, D8, D9: CatNo (none) -> 1516-QBL7IW60D-NW-ND
- D11, D12: CatNo (none) -> 732-5016-ND
- D21, D22, D23, D24, D25, D26, D27, D28, D29, D30, D31, D32, D33, D34, D35, D36, D37, D38, D39, D40: CatNo (none) -> 3147-B1A81NG--20C000313U1930CT-ND
- D41, D42, D43, D44, D45, D46, D47, D48, D49, D50, D51, D52, D53, D54, D55, D56, D57, D58, D59, D60, D61, D62, D63, D64, D65, D66, D67, D68, D69, D70: CatNo (none) -> 3147-B1A81NB--20C000313U1930CT-ND
- U1: CatNo (none) -> ICM7218AIQI+-ND
Other:
- note added: "CONTROL BITS ID4 - ~{SHUTDOWN} ID5 - ~{DECODE} ID6 - HEX/~{CODEB} ID7 - DATA COMING"
