File: KiCAD/ControlPanelRTC/ControlPanelRTC.kicad_sch (KiCad schematic)
At the start: 22 parts, among them J1 Conn_01x04_Pin, J2 Conn_01x04_Pin, Q1 TEPT4400, SW1 SW_Push, SW2 SW_Push, SW3 SW_Push, SW4 SW_Push, U1 DS3231MZ

Commit message: readme
Other:
- note added: "Real-time Clock"
- note added: "UART link to main PCB"
Changed lines of the file:
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@@
 	(generator_version "9.0")
 	(paper "A4")
+	(text "UART link\nto main PCB"
+		(exclude_from_sim no)
+		(at 153.416 29.464 0)
+		(effects
+			(font
+				(size 1.905 1.905)
+			)
+		)
+	)
 	(text "I2C DISPLAY"
 		(exclude_from_sim no)
-		(at 53.34 55.88 0)
+		(at 63.246 43.434 0)
 		(effects
 			(font
-				(size 1.27 1.27)
+				(size 1.905 1.905)
 			)
 		)
+	)
+	(text "Real-time Clock"
+		(exclude_from_sim no)
+		(at 61.722 105.918 0)
+		(effects
+			(font
+				(size 1.905 1.905)
+			)
+		)

Commit message: work on control panel
Parts:
- removed A1: Arduino_Nano_v3.x, Module:Arduino_Nano, symbol MCU_Module:Arduino_Nano_v3.x
- removed J1: Conn_01x04_Pin, Connector_PinHeader_2.54mm:PinHeader_1x04_P2.54mm_Vertical, symbol Connector:Conn_01x04_Pin
- added C3: 10uF, Capacitor_SMD:C_1206_3216Metric_Pad1.33x1.80mm_HandSolder, symbol Device:C
- added C4: 22uF, Capacitor_SMD:C_1206_3216Metric_Pad1.33x1.80mm_HandSolder, symbol Device:C
- added C5, C6: 0.1uF, Capacitor_SMD:C_1206_3216Metric_Pad1.33x1.80mm_HandSolder, symbol Device:C
- added J1, J3: Conn_01x05, Connector_PinHeader_2.54mm:PinHeader_1x04_P2.54mm_Horizontal, symbol Connector_Generic:Conn_01x04
- added J4: AVR-ISP-6, Connector_PinHeader_2.54mm:PinHeader_2x03_P2.54mm_Horizontal, symbol Connector:AVR-ISP-6
- added R4: 4.7k, Resistor_SMD:R_1206_3216Metric, symbol Device:R_US
- added U2: AZ1117-3.3, Package_TO_SOT_SMD:SOT-223-3_TabPin2, symbol Regulator_Linear:AZ1117-3.3
- added U3: ATmega328P-P, Package_QFP:TQFP-32_7x7mm_P0.8mm, symbol MCU_Microchip_ATmega:ATmega328P-A
- BT1: footprint Battery:BatteryHolder_Keystone_103_1x20mm -> Battery:BatteryHolder_Keystone_3000_1x12mm
- R1, R2, R3: value R_US -> 4.7k
- R6, R7: value R_US -> 1k
- SW1, SW2, SW3, SW4: footprint AA_parts:Push_SW -> AA_parts:SW4_1825910-B_TEC; symbol Switch:SW_Push -> my_sw:SW_Push_pins13
Connections:
- net GND: now also SW1.3, SW2.3, SW3.3, SW4.3, C3.2, C4.2, C5.2, C6.2, J1.4 (Pin_4), J3.2 (Pin_2), J3.3 (Pin_3), J4.6 (GND), U2.1 (GND), U3.21 (GND), U3.3 (GND), U3.5 (GND); no longer SW1.2, SW2.2, SW3.2, SW4.2
- net S0: now also U3.23 (PC0)
- net S1: now also U3.24 (PC1)
- net S2: now also U3.25 (PC2)
- net S3: now also U3.26 (PC3)
- net SCL: now also U3.28 (PC5)
- net SDA: now also U3.27 (PC4)
- net VCC: now also C3.1, C5.1, C6.1, J1.1 (Pin_1), J3.4 (Pin_4), J4.2 (VCC), R4.1, U2.3 (VI), U3.18 (AVCC), U3.20 (AREF), U3.4 (VCC), U3.6 (VCC)
- net at R6.1: now also J1.2 (Pin_2)
- net at R7.1: now also J1.3 (Pin_3)
- net TXD: now reaches R6.2
- net TXD: now also U3.31 (PD1)
- net RXD: now reaches R7.2
- net RXD: now also U3.30 (PD0)
- net ALS renamed A0
- net A0: now also U3.19 (ADC6)
- new net +3.3V: C4.1, J3.1 (Pin_1), U2.2 (VO)
- new net MISO: J4.1 (MISO), U3.16 (PB4)
- new net MOSI: J4.4 (MOSI), U3.15 (PB3)
- new net SCK: J4.3 (SCK), U3.17 (PB5)
- new net ~{RESET}: J4.5 (~{RST}), R4.2, U3.29 (~{RESET}/PC6)
Other:
- moved on the sheet: H1, H2, H3, H4, R6, R7, SW1, SW2, SW3, SW4
